File: MouseWB5/_autosave-MouseWB5.kicad_sch (KiCad schematic)
At the start: 68 parts, among them J1 USB_C_Receptacle_USB2.0_14P, J10 Conn_01x09_Socket, J2 Conn_01x11_Socket, J3 Conn_01x09_Socket, J4 Conn_01x02_Socket, J5 Conn_01x02_Socket, J6 Conn_01x02_Socket, J7 Conn_01x02_Socket, J8 Conn_01x02_Socket, J9 Conn_01x02_Socket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

Commit message: work
Parts:
- J10, J3: footprint (none) -> Connector_PinHeader_1.00mm:PinHeader_1x09_P1.00mm_Vertical
- J2: footprint (none) -> Connector_PinHeader_1.00mm:PinHeader_1x11_P1.00mm_Vertical
Changed lines of the file:
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@@
 			)
 		)
-		(property "Footprint" ""
+		(property "Footprint" "Connector_PinHeader_1.00mm:PinHeader_1x09_P1.00mm_Vertical"
 			(at 331.47 181.61 0)
 			(effects
@@
 			)
 		)
-		(property "Footprint" ""
+		(property "Footprint" "Connector_PinHeader_1.00mm:PinHeader_1x11_P1.00mm_Vertical"
 			(at 331.47 119.38 0)
 			(effects
@@
 			)
 		)
-		(property "Footprint" ""
+		(property "Footprint" "Connector_PinHeader_1.00mm:PinHeader_1x09_P1.00mm_Vertical"
 			(at 331.47 149.86 0)
 			(effects
