File: MouseWB5/MouseWB5.kicad_pcb (KiCad board)
At the start: 6 copper layers, 65.5 x 40 mm, 66 parts, among them J1 USB_C_Receptacle_USB2.0_14P, J10 Conn_01x09_Socket, J11 TC2030, J2 Conn_01x11_Socket, J3 Conn_01x09_Socket, J8 Conn_01x02_Socket, J9 Conn_01x02_Socket, M1 Conn_01x02_Socket, M2 Conn_01x02_Socket, M3 Conn_01x02_Socket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

Commit message: work
Routing:
- net +1V8: track 90.9 -> 92.9 mm
- net GND: vias 27 -> 23
Changed lines of the file:
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@@
-	)
-	(via
-		(at 123.5 115)
-		(size 0.6)
-		(drill 0.3)
-		(layers "F.Cu" "B.Cu")
-		(net 81)
 	)
 	(via
@@
 	)
 	(via
-		(at 143.75 125.5)
-		(size 0.6)
-		(drill 0.3)
-		(layers "F.Cu" "B.Cu")
-		(net 81)
-	)
-	(via
 		(at 142 103.5)
 		(size 0.6)
@@
 	)
 	(via
-		(at 123.5 123.5)
-		(size 0.6)
-		(drill 0.3)
-		(layers "F.Cu" "B.Cu")
-		(net 81)
-	)
-	(via
 		(at 128.25 138.5)
 		(size 0.6)
@@
 	)
 	(via
-		(at 101 113.75)
+		(at 101 114.25)
 		(size 0.6)
 		(drill 0.3)
@@
 	(via
 		(at 110.25 123.25)
-		(size 0.6)
-		(drill 0.3)
-		(layers "F.Cu" "B.Cu")
-		(net 81)
-	)
-	(via
-		(at 143.5 115)
 		(size 0.6)
 		(drill 0.3)
@@
 	)
 	(segment
-		(start 118.5 116)
-		(end 116.25 118.25)
+		(start 116.25 117)
+		(end 124 109.25)
 		(width 0.5)
 		(layer "F.Cu")
@@
 	)
 	(segment
-		(start 138.1485 110.75)
-		(end 129.75 110.75)
+		(start 124 109.25)
+		(end 135.25 109.25)
 		(width 0.5)
 		(layer "F.Cu")
@@
 	)
 	(segment
+		(start 146 120)
+		(end 157 120)
+		(width 0.5)
+		(layer "F.Cu")
+		(net 141)
+	)
+	(segment
 		(start 114.512075 124.55)
+		(end 116.25 122.812075)
+		(width 0.5)
+		(layer "F.Cu")
+		(net 141)
+	)
+	(segment
+		(start 135.25 109.25)
+		(end 146 120)
+		(width 0.5)
+		(layer "F.Cu")
+		(net 141)
+	)
+	(segment
+		(start 113.5635 124.6135)
 		(end 113.5635 124.55)
 		(width 0.5)
@@
 	)
 	(segment
-		(start 116.25 122.812075)
+		(start 113.5635 124.55)
 		(end 114.512075 124.55)
 		(width 0.5)
@@
 	)
 	(segment
-		(start 160 123)
-		(end 157 120)
-		(width 0.5)
-		(layer "F.Cu")
-		(net 141)
-	)
-	(segment
-		(start 116.25 118.25)
-		(end 116.25 122.812075)
-		(width 0.5)
-		(layer "F.Cu")
-		(net 141)
-	)
-	(segment
-		(start 124.5 116)
-		(end 118.5 116)
-		(width 0.5)
-		(layer "F.Cu")
-		(net 141)
-	)
-	(segment
-		(start 162.5 123)
+		(start 157 120)
 		(end 160 123)
 		(width 0.5)
@@
 	)
 	(segment
-		(start 113.5635 124.55)
-		(end 113.5635 124.6135)
+		(start 116.25 122.812075)
+		(end 116.25 117)
 		(width 0.5)
 		(layer "F.Cu")
@@
 	)
 	(segment
-		(start 129.75 110.75)
-		(end 124.5 116)
+		(start 160 123)
+		(end 162.5 123)
 		(width 0.5)
 		(layer "F.Cu")
-		(net 141)
-	)
-	(segment
-		(start 147.3985 120)
-		(end 138.1485 110.75)
-		(width 0.5)
-		(layer "F.Cu")
-		(net 141)
-	)
-	(segment
-		(start 157 120)
-		(end 147.3985 120)
-		(width 0.5)
-		(layer "F.Cu")

Commit message: work
Parts:
- added Q1: FDN327N, FDN327N:SSOT-3, F.Cu at (144.2, 120.0)
- moved MR3 0.26 mm to (116.5, 108.2)
- moved MR4 0.25 mm to (118.0, 108.3)
Routing:
- net +1V8: track 92.9 -> 89.3 mm
Changed lines of the file:
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@@
 	(net 162 "unconnected-(J10-Pin_7-Pad7)")
 	(net 163 "unconnected-(J10-Pin_5-Pad5)")
+	(net 164 "unconnected-(Q1-Pad3)")
+	(net 165 "unconnected-(Q1-Pad2)")
+	(net 166 "unconnected-(Q1-Pad1)")
 	(footprint "MountingHole:MountingHole_2.1mm"
 		(layer "F.Cu")
@@
 	(footprint "Resistor_SMD:R_0402_1005Metric"
 		(layer "F.Cu")
-		(at 116.5 107.99 90)
+		(at 116.5 108.25 90)
 		(descr "Resistor SMD 0402 (1005 Metric), square (rectangular) end terminal, IPC_7351 nominal, (Body size source: IPC-SM-782 page 72, https://www.pcb-3d.com/wordpress/wp-content/uploads/ipc-sm-782a_amendment_1_and_2.pdf), generated with kicad-footprint-generator")
 		(tags "resistor")
@@
 	(footprint "Resistor_SMD:R_0402_1005Metric"
 		(layer "F.Cu")
-		(at 118 108.01 90)
+		(at 118 108.26 90)
 		(descr "Resistor SMD 0402 (1005 Metric), square (rectangular) end terminal, IPC_7351 nominal, (Body size source: IPC-SM-782 page 72, https://www.pcb-3d.com/wordpress/wp-content/uploads/ipc-sm-782a_amendment_1_and_2.pdf), generated with kicad-footprint-generator")
 		(tags "resistor")
@@
 		)
 	)
+	(footprint "FDN327N:SSOT-3"
+		(layer "F.Cu")
+		(at 144.25 120 -90)
+		(descr "SuperSOT-3")
+		(property "Reference" "Q1"
+			(at 3.815515 -1.780575 90)
+			(layer "F.SilkS")
+			(hide yes)
+			(effects
+				(font
+					(size 0.801157 0.801157)
+					(thickness 0.15)
+				)
+			)
+		)
+		(property "Value" "FDN327N"
+			(at 0.53364 2.769855 90)
+			(layer "F.Fab")
+			(hide yes)
+			(effects
+				(font
+					(size 0.640291 0.640291)
+					(thickness 0.15)
+				)
+			)
+		)
+		(property "Datasheet" ""
+			(at 0 0 90)
+			(layer "F.Fab")
+			(hide yes)
+			(effects
+				(font
+					(size 1.27 1.27)
+					(thickness 0.15)
+				)
+			)
+		)
+		(property "Description" ""
+			(at 0 0 90)
+			(layer "F.Fab")
+			(hide yes)
+			(effects
+				(font
+					(size 1.27 1.27)
+					(thickness 0.15)
+				)
+			)
+		)
+		(sheetname "/")
+		(sheetfile "MouseWB5.kicad_sch")
+		(attr smd)
+		(fp_line
+			(start -1.4224 0.1524)
+			(end -1.4224 -0.6604)
+			(stroke
+				(width 0.2032)
+				(type solid)
+			)
+			(layer "F.SilkS")
+		)
+		(fp_line
+			(start -1.4224 -0.6604)
+			(end -0.7636 -0.6604)
+			(stroke
+				(width 0.2032)
+				(type solid)
+			)
+			(layer "F.SilkS")
+		)
+		(fp_line
+			(start 0.7636 -0.6604)
+			(end 1.4224 -0.6604)
+			(stroke
+				(width 0.2032)
+				(type solid)
+			)
+			(layer "F.SilkS")
+		)
+		(fp_line
+			(start 1.4224 -0.6604)
+			(end 1.4224 0.1524)
+			(stroke
+				(width 0.2032)
+				(type solid)
+			)
+			(layer "F.SilkS")
+		)
+		(fp_line
+			(start -1.4224 0.6604)
+			(end -1.4224 -0.6604)
+			(stroke
+				(width 0.2032)
+				(type solid)
+			)
+			(layer "F.Fab")
+		)
+		(fp_line
+			(start 1.4224 0.6604)
+			(end -1.4224 0.6604)
+			(stroke
+				(width 0.2032)
+				(type solid)
+			)
+			(layer "F.Fab")
+		)
+		(fp_line
+			(start -1.4224 -0.6604)
+			(end 1.4224 -0.6604)
+			(stroke
+				(width 0.2032)
+				(type solid)
+			)
+			(layer "F.Fab")
+		)
+		(fp_line
+			(start 1.4224 -0.6604)
+			(end 1.4224 0.6604)
+			(stroke
+				(width 0.2032)
+				(type solid)
+			)
+			(layer "F.Fab")
+		)
+		(fp_poly
+			(pts
+				(xy -1.17065 0.7112) (xy -0.7112 0.7112) (xy -0.7112 1.2979) (xy -1.17065 1.2979)
+			)
+			(stroke
+				(width 0.01)
+				(type solid)
+			)
+			(fill yes)
+			(layer "F.Fab")
+		)
+		(fp_poly
+			(pts
+				(xy 0.712299 0.7112) (xy 1.1684 0.7112) (xy 1.1684 1.2974) (xy 0.712299 1.2974)
+			)
+			(stroke
+				(width 0.01)
+				(type solid)
+			)
+			(fill yes)
+			(layer "F.Fab")
+		)
+		(fp_poly
+			(pts
+				(xy -0.22891 -1.2954) (xy 0.2286 -1.2954) (xy 0.2286 -0.712165) (xy -0.22891 -0.712165)
+			)
+			(stroke
+				(width 0.01)
+				(type solid)
+			)
+			(fill yes)
+			(layer "F.Fab")
+		)
+		(pad "1" smd rect
+			(at -0.95 1.1 270)
+			(size 1 1.4)
+			(layers "F.Cu" "F.Mask" "F.Paste")
+			(net 166 "unconnected-(Q1-Pad1)")
+			(pintype "passive")
+			(solder_mask_margin 0.102)
+		)
+		(pad "2" smd rect
+			(at 0.95 1.1 270)
+			(size 1 1.4)
+			(layers "F.Cu" "F.Mask" "F.Paste")
+			(net 165 "unconnected-(Q1-Pad2)")
+			(pintype "passive")
+			(solder_mask_margin 0.102)
+		)
+		(pad "3" smd rect
+			(at 0 -1.1 270)
+			(size 1 1.4)
+			(layers "F.Cu" "F.Mask" "F.Paste")
+			(net 164 "unconnected-(Q1-Pad3)")
+			(pintype "passive")
+			(solder_mask_margin 0.102)
+		)
+		(embedded_fonts no)
+	)
 	(footprint "Connector_JST:JST_EH_B2B-EH-A_1x02_P2.50mm_Vertical"
 		(layer "F.Cu")
@@
 	)
 	(segment
-		(start 116.25 117)
-		(end 124 109.25)
+		(start 119.75 108.75)
+		(end 147.25 108.75)
 		(width 0.5)
 		(layer "F.Cu")
@@
 	)
 	(segment
-		(start 124 109.25)
-		(end 135.25 109.25)
+		(start 116.25 112.25)
+		(end 119.75 108.75)
 		(width 0.5)
 		(layer "F.Cu")
@@
 	)
 	(segment
-		(start 146 120)
-		(end 157 120)
+		(start 113.5635 124.55)
+		(end 114.512075 124.55)
 		(width 0.5)
 		(layer "F.Cu")
@@
 	)
 	(segment
-		(start 135.25 109.25)
-		(end 146 120)
-		(width 0.5)
-		(layer "F.Cu")
-		(net 141)
-	)
-	(segment
-		(start 113.5635 124.6135)
-		(end 113.5635 124.55)
+		(start 116.25 122.812075)
+		(end 116.25 112.25)
 		(width 0.5)
 		(layer "F.Cu")
@@
 	)
 	(segment
-		(start 113.5635 124.55)
-		(end 114.512075 124.55)
+		(start 147.25 108.75)
+		(end 149.25 110.75)
 		(width 0.5)
 		(layer "F.Cu")
@@
 	)
 	(segment
-		(start 157 120)
-		(end 160 123)
+		(start 149.25 110.75)
+		(end 160.171572 110.75)
 		(width 0.5)
 		(layer "F.Cu")
@@
 	)
 	(segment
-		(start 116.25 122.812075)
-		(end 116.25 117)
+		(start 160.171572 110.75)
+		(end 160.585786 110.335786)
 		(width 0.5)
 		(layer "F.Cu")
@@
 	)
 	(segment
-		(start 160 123)
-		(end 162.5 123)
+		(start 113.5635 124.6135)
+		(end 113.5635 124.55)
 		(width 0.5)
 		(layer "F.Cu")

Commit message: work
Parts:
- moved H3 2.02 mm to (140.2, 127.5)
- moved H2 1.03 mm to (125.2, 112.5)
Connections:
- Q1 pad 1: unconnected-(Q1-Pad1) -> /FAN_CTRL
Other:
- outline, holes or cut-outs redrawn
Changed lines of the file:
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@@
 	(net 164 "unconnected-(Q1-Pad3)")
 	(net 165 "unconnected-(Q1-Pad2)")
-	(net 166 "unconnected-(Q1-Pad1)")
+	(net 166 "/FAN_CTRL")
 	(footprint "MountingHole:MountingHole_2.1mm"
 		(layer "F.Cu")
-		(at 142 128.5 90)
+		(at 140.25 127.5 90)
 		(descr "Mounting Hole 2.1mm, no annular")
 		(tags "mounting hole 2.1mm no annular")
@@
 			(size 1 1.4)
 			(layers "F.Cu" "F.Mask" "F.Paste")
-			(net 166 "unconnected-(Q1-Pad1)")
+			(net 166 "/FAN_CTRL")
 			(pintype "passive")
 			(solder_mask_margin 0.102)
@@
 	(footprint "MountingHole:MountingHole_2.1mm"
 		(layer "F.Cu")
-		(at 125 111.5 90)
+		(at 125.25 112.5 90)
 		(descr "Mounting Hole 2.1mm, no annular")
 		(tags "mounting hole 2.1mm no annular")
@@
 	)
 	(gr_line
-		(start 143 127.5)
+		(start 143 129.5)
 		(end 143 121.25)
 		(stroke
@@
 	)
 	(gr_circle
-		(center 133.5 120)
-		(end 141.5 120)
+		(center 132.75 120)
+		(end 140.75 120)
 		(stroke
 			(width 0.05)
-			(type default)
+			(type solid)
 		)
 		(fill no)

Commit message: work
Connections:
- U1 pad 28: unconnected-(U1-PA10-Pad28) -> VBUS

Commit message: work
Parts:
- moved U7 37.9 mm to (115.5, 116.3), turned to 180 degrees
- moved C10 36.9 mm to (113.8, 112.5), turned to -90 degrees
- moved C2 1.00 mm to (118.2, 120.0)
- moved U5 1.00 mm to (120.8, 120.0), turned to 0 degrees
Connections:
- J10 pad 2: +3V3 -> +1V8
- J10 pad 3: +1V8 -> +3V3
- J2 pad 2: +3V3 -> +1V8
- J2 pad 3: +1V8 -> +3V3
- J3 pad 2: +3V3 -> +1V8
- J3 pad 3: +1V8 -> +3V3
- U1 pad 32: +1V8 -> +3V3
Routing:
- net +3V3: track 43.3 -> 83.1 mm
- net +BATT: track 206.2 -> 200.2 mm, vias 21 -> 20
- net GND: track 31.6 -> 28.5 mm, vias 23 -> 22
- net +1V8: track 89.3 -> 90.9 mm

Commit message: work
Parts:
- moved Q1 8.14 mm to (152.0, 122.5)
Routing:
- net +BATT: track 200.2 -> 205.0 mm, vias 20 -> 21
- net GND: track 28.5 -> 33.2 mm, vias 22 -> 23
- net /CHARGE: track 0.00 -> 0.89 mm, vias 0 -> 1
- net /PWRON: track 0.00 -> 0.87 mm, vias 0 -> 1
Other:
- board text added: "NMOS"
Changed lines of the file:
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@@
 	(footprint "FDN327N:SSOT-3"
 		(layer "F.Cu")
-		(at 144.25 120 -90)
+		(at 152 122.5 -90)
 		(descr "SuperSOT-3")
 		(property "Reference" "Q1"
@@
 		(layer "B.SilkS")
 	)
+	(gr_rect
+		(start 150 120.75)
+		(end 154 124.25)
+		(stroke
+			(width 0.1)
+			(type default)
+		)
+		(fill no)
+		(layer "B.SilkS")
+	)
 	(gr_arc
 		(start 101.5 135.5)
@@
 		)
 	)
+	(gr_text "NMOS"
+		(at 151.75 123.625 270)
+		(layer "B.SilkS")
+		(effects
+			(font
+				(size 0.5 0.5)
+				(thickness 0.125)
+				(bold yes)
+			)
+			(justify left bottom mirror)
+		)
+	)
 	(gr_text "I2C0"
 		(at 157.75 130.75 225)
@@
 	)
 	(segment
-		(start 111.725 123.25)
-		(end 111.725 122.7855)
-		(width 0.3)
-		(layer "F.Cu")
-		(net 73)
-	)
-	(segment
 		(start 154.5 116.65)
 		(end 153.75 116.65)
@@
 	)
 	(segment
-		(start 114.6798 122)
-		(end 113.75 122)
-		(width 0.3)
-		(layer "F.Cu")
-		(net 73)
-	)
-	(segment
-		(start 111.725 122.7855)
-		(end 112.5105 122)
-		(width 0.3)
-		(layer "F.Cu")
-		(net 73)
-	)
-	(segment
 		(start 153.75 118)
 		(end 153.75 116.65)
@@
 	)
 	(segment
-		(start 114.9048 121.775)
-		(end 114.6798 122)
-		(width 0.3)
-		(layer "F.Cu")
-		(net 73)
-	)
-	(segment
 		(start 133.75 102.2)
 		(end 134.45 101.5)
@@
 	)
 	(segment
-		(start 114.9048 121.25)
-		(end 114.9048 121.775)
+		(start 101.9249 105.4249)
+		(end 101.9249 105.65766)
 		(width 0.3)
 		(layer "F.Cu")
@@
 	)
 	(segment
-		(start 101.9249 105.4249)
-		(end 101.9249 105.65766)
+		(start 111.1865 123.5635)
+		(end 111.5 123.25)
 		(width 0.3)
 		(layer "F.Cu")
@@
 	)
 	(segment
-		(start 111.1865 123.5635)
-		(end 111.5 123.25)
+		(start 112.2605 122.25)
+		(end 114.4298 122.25)
 		(width 0.3)
 		(layer "F.Cu")
@@
 	)
 	(segment
+		(start 114.4298 122.25)
+		(end 114.9048 121.775)
+		(width 0.3)
+		(layer "F.Cu")
+		(net 73)
+	)
+	(segment
 		(start 101.9249 135.65766)
 		(end 101.9249 135.4249)
@@
 	)
 	(segment
-		(start 111.5 123.25)
-		(end 111.725 123.25)
+		(start 114.074 116.573999)
+		(end 114.074 115.801)
+		(width 0.3)
+		(layer "F.Cu")
+		(net 73)
+	)
+	(segment
+		(start 114.25 115.625)
+		(end 113.875 115.625)
 		(width 0.3)
 		(layer "F.Cu")
@@
 	)
 	(segment
-		(start 112.5105 122)
-		(end 113.75 122)
+		(start 111.5 123.25)
+		(end 111.725 123.25)
 		(width 0.3)
 		(layer "F.Cu")
@@
 	)
 	(segment
+		(start 114.425001 116.925)
+		(end 114.074 116.573999)
+		(width 0.3)
+		(layer "F.Cu")
+		(net 73)
+	)
+	(segment
 		(start 155.75 118)
 		(end 155.75 116.75)
@@
 	)
 	(segment
+		(start 111.725 123.25)
+		(end 111.725 122.7855)
+		(width 0.3)
+		(layer "F.Cu")
+		(net 73)
+	)
+	(segment
 		(start 111.725 124.55)
 		(end 111.54343 124.55)
@@
 	)
 	(segment
+		(start 113.875 115.625)
+		(end 113.75 115.75)
+		(width 0.3)
+		(layer "F.Cu")
+		(net 73)
+	)
+	(segment
 		(start 111.5 110.75)
 		(end 111.5 111.55)
@@
 	)
 	(segment
+		(start 114.074 115.801)
+		(end 114.25 115.625)
+		(width 0.3)
+		(layer "F.Cu")
+		(net 73)
+	)
+	(segment
 		(start 101.9249 102.1749)
 		(end 101.9249 102.40766)
@@
 	)
 	(segment
+		(start 114.9048 121.775)
+		(end 114.9048 121.25)
+		(width 0.3)
+		(layer "F.Cu")
+		(net 73)
+	)
+	(segment
+		(start 114.6125 115.625)
+		(end 114.25 115.625)
+		(width 0.3)
+		(layer "F.Cu")
+		(net 73)
+	)
+	(segment
+		(start 111.725 122.7855)
+		(end 112.2605 122.25)
+		(width 0.3)
+		(layer "F.Cu")
+		(net 73)
+	)
+	(segment
 		(start 135.75 101.75)
 		(end 134.7 101.75)
@@
 	)
 	(segment
+		(start 114.6125 116.925)
+		(end 114.425001 116.925)
+		(width 0.3)
+		(layer "F.Cu")
+		(net 73)
+	)
+	(segment
 		(start 101.9249 112.4249)
 		(end 101.9249 112.835006)
@@
 	)
 	(via
+		(at 113.75 115.75)
+		(size 0.6)
+		(drill 0.3)
+		(layers "F.Cu" "B.Cu")
+		(net 73)
+	)
+	(via
 		(at 135.75 101.75)
 		(size 0.6)
@@
 	)
 	(segment
+		(start 111.5 110.75)
+		(end 111.5 115.75)
+		(width 0.6)
+		(layer "B.Cu")
+		(net 73)
+	)
+	(segment
 		(start 144.75 129.75)
 		(end 140.5 134)
@@
 	)
 	(segment
-		(start 111.5 110.75)
+		(start 111.5 115.75)
 		(end 111.5 121.75)
 		(width 0.6)
@@
 	)
 	(segment
+		(start 111.5 115.75)
+		(end 113.75 115.75)
+		(width 0.6)
+		(layer "B.Cu")
+		(net 73)
+	)
+	(segment
 		(start 102 105.5)
 		(end 102 105.75)
@@
 	)
 	(segment
-		(start 101.0751 136.8251)
-		(end 101 136.75)
+		(start 112.76 115.75)
+		(end 112.76 118.24)
 		(width 0.3)
 		(layer "F.Cu")
@@
 	)
 	(segment
-		(start 114.75 123.25)
-		(end 114 122.5)
+		(start 101.0751 136.8251)
+		(end 101 136.75)
 		(width 0.3)
 		(layer "F.Cu")
@@
 	)
 	(segment
+		(start 112.76 115.75)
+		(end 112.76 117.5)
+		(width 0.3)
+		(layer "F.Cu")
+		(net 80)
+	)
+	(segment
 		(start 101.0751 106.8251)
 		(end 101 106.75)
@@
 	)
 	(segment
+		(start 112.76 118.24)
+		(end 112.75 118.25)
+		(width 0.3)
+		(layer "F.Cu")
+		(net 80)
+	)
+	(segment
 		(start 104.336775 100.8)
 		(end 105.23 101.693225)
@@
 	)
 	(segment
-		(start 112.6125 122.8875)
-		(end 112.6125 123.9)
+		(start 101.0751 111.5751)
+		(end 101.0751 110.3251)
 		(width 0.3)
 		(layer "F.Cu")
@@
 	)
 	(segment
-		(start 101.0751 111.5751)
-		(end 101.0751 110.3251)
+		(start 112.76 115)
+		(end 112.76 115.75)
 		(width 0.3)
 		(layer "F.Cu")
@@
 	)
 	(segment
-		(start 114 122.5)
-		(end 113 122.5)
+		(start 112.75 119.597599)
+		(end 113.4524 120.299999)
+		(width 0.3)
+		(layer "F.Cu")
+		(net 80)
+	)
+	(segment
+		(start 112.75 118.25)
+		(end 112.75 119.597599)
 		(width 0.3)
 		(layer "F.Cu")
@@
 	)
 	(segment
+		(start 114.6125 116.275)
+		(end 115.5 116.275)
+		(width 0.3)
+		(layer "F.Cu")
+		(net 80)
+	)
+	(segment
 		(start 133.25 102.2)
 		(end 132.55 101.5)
@@
 	)
 	(segment
-		(start 113 122.5)
-		(end 112.6125 122.8875)
-		(width 0.3)
-		(layer "F.Cu")
-		(net 80)
-	)
-	(segment
 		(start 133.75 136.4875)
 		(end 133.75 137.8)
@@
 	)
 	(via
-		(at 114.75 123.25)
+		(at 115.25 123.25)
 		(size 0.6)
 		(drill 0.3)
@@
 	)
 	(via
+		(at 112.75 118.25)
+		(size 0.6)
+		(drill 0.3)
+		(layers "F.Cu" "B.Cu")
+		(net 80)
+	)
+	(via
 		(at 102.75 100.8)
 		(size 0.6)
@@
 	)
 	(segment
+		(start 115.700001 120.299999)
+		(end 115.75 120.25)
+		(width 0.2)
+		(layer "F.Cu")
+		(net 131)
+	)
+	(segment
+		(start 114.9048 120.299999)
+		(end 115.700001 120.299999)
+		(width 0.2)
+		(layer "F.Cu")
+		(net 131)
+	)
+	(via
+		(at 115.75 120.25)
+		(size 0.6)
+		(drill 0.3)
+		(layers "F.Cu" "B.Cu")
+		(net 131)
+	)
+	(segment
+		(start 115.650002 119.349998)
+		(end 115.75 119.25)
+		(width 0.2)
+		(layer "F.Cu")
+		(net 132)
+	)
+	(segment
+		(start 114.9048 119.349998)
+		(end 115.650002 119.349998)
+		(width 0.2)
+		(layer "F.Cu")
+		(net 132)
+	)
+	(via
+		(at 115.75 119.25)
+		(size 0.6)
+		(drill 0.3)
+		(layers "F.Cu" "B.Cu")
+		(net 132)
+	)
+	(segment

Commit message: work
Routing:
- net GND: vias 23 -> 24
Changed lines of the file:
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@@
+	)
+	(via
+		(at 120.75 120)
+		(size 0.6)
+		(drill 0.3)
+		(layers "F.Cu" "B.Cu")
+		(free yes)
+		(net 80)
 	)
 	(via

Commit message: work
Routing:
- net VBUS: track 10.3 -> 19.0 mm
- net +3V3: track 83.1 -> 85.8 mm
- net /USB_D-: track 0.00 -> 1.35 mm
- net /USB_D+: track 0.00 -> 1.34 mm
- net GND: track 33.2 -> 33.9 mm, vias 24 -> 25
Changed lines of the file:
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@@
+	)
+	(segment
+		(start 105.75 123.25)
+		(end 106.786 122.214)
+		(width 0.2)
+		(layer "F.Cu")
+		(net 79)
+	)
+	(segment
+		(start 108.309 122.214)
+		(end 108.545 122.45)
+		(width 0.2)
+		(layer "F.Cu")
+		(net 79)
+	)
+	(segment
+		(start 105.75 125)
+		(end 105.75 123.25)
+		(width 0.2)
+		(layer "F.Cu")
+		(net 79)
 	)
 	(segment
@@
 	)
 	(segment
+		(start 104.875 128.325)
+		(end 104.875 127.875)
+		(width 0.2)
+		(layer "F.Cu")
+		(net 79)
+	)
+	(segment
+		(start 105.25 125.5)
+		(end 105.75 125)
+		(width 0.2)
+		(layer "F.Cu")
+		(net 79)
+	)
+	(segment
+		(start 105.25 127.5)
+		(end 105.25 125.5)
+		(width 0.2)
+		(layer "F.Cu")
+		(net 79)
+	)
+	(segment
+		(start 104.875 127.875)
+		(end 105.25 127.5)
+		(width 0.2)
+		(layer "F.Cu")
+		(net 79)
+	)
+	(segment
+		(start 106.786 122.214)
+		(end 108.309 122.214)
+		(width 0.2)
+		(layer "F.Cu")
+		(net 79)
+	)
+	(segment
 		(start 110.3 122.45)
 		(end 111.5 121.25)
@@
 	)
 	(segment
+		(start 103.5 128.325)
+		(end 103.5 127.75)
+		(width 0.2)
+		(layer "F.Cu")
+		(net 80)
+	)
+	(segment
 		(start 102.75 100.8)
 		(end 104.336775 100.8)
@@
 		(end 101 136.75)
 		(width 0.3)
+		(layer "F.Cu")
+		(net 80)
+	)
+	(segment
+		(start 103.5 127.75)
+		(end 103.375 127.75)
+		(width 0.2)
 		(layer "F.Cu")
 		(net 80)
@@
 	)
 	(via
+		(at 103.375 127.75)
+		(size 0.6)
+		(drill 0.3)
+		(layers "F.Cu" "B.Cu")
+		(net 80)
+	)
+	(via
 		(at 142 103.5)
 		(size 0.6)
@@
 	)
 	(segment
+		(start 103.05 128.8)
+		(end 102.5 128.25)
+		(width 0.2)
+		(layer "F.Cu")
+		(net 81)
+	)
+	(segment
 		(start 117.25 116.5)
 		(end 116.825 116.925)
@@
 	)
 	(segment
+		(start 102.5 128.25)
+		(end 102.5 126.75)
+		(width 0.2)
+		(layer "F.Cu")
+		(net 81)
+	)
+	(segment
 		(start 117.25 114.75)
 		(end 117.25 116.5)
@@
 	)
 	(segment
+		(start 103.5 128.8)
+		(end 103.05 128.8)
+		(width 0.2)
+		(layer "F.Cu")
+		(net 81)
+	)
+	(segment
 		(start 116.825 116.925)
 		(end 116.451 116.925)
@@
 		(layer "F.Cu")
 		(net 82)
+	)
+	(segment
+		(start 104.425 128.325)
+		(end 104.425 127.27)
+		(width 0.2)
+		(layer "F.Cu")
+		(net 83)
+	)
+	(segment
+		(start 104.425 127.27)
+		(end 104.625 127.07)
+		(width 0.2)
+		(layer "F.Cu")
+		(net 83)
+	)
+	(segment
+		(start 103.975 128.325)
+		(end 103.975 127.295)
+		(width 0.2)
+		(layer "F.Cu")
+		(net 84)
+	)
+	(segment
+		(start 103.975 127.295)
+		(end 103.75 127.07)
+		(width 0.2)
+		(layer "F.Cu")
+		(net 84)
 	)
 	(segment
@@
 	)
 	(segment
-		(start 104.625 126.43)
-		(end 104.625 125.875)
+		(start 105.251 124.731016)
+		(end 104.866009 125.116009)
 		(width 0.3)
 		(layer "F.Cu")
@@
 	)
 	(segment
-		(start 105.75 122.5)
-		(end 105.75 124.75)
+		(start 104.625 125.357016)
+		(end 104.625 126.43)
 		(width 0.3)
 		(layer "F.Cu")
@@
 	)
 	(segment
-		(start 107.5 120.75)
-		(end 105.75 122.5)
+		(start 104.866009 125.116009)
+		(end 104.625 125.357016)
 		(width 0.3)
 		(layer "F.Cu")
@@
 	)
 	(segment
-		(start 108.545 120.75)
-		(end 107.5 120.75)
+		(start 105.251 122.95752)
+		(end 105.251 124.731016)
+		(width 0.3)
+		(layer "F.Cu")
+		(net 118)
+	)
+	(segment
+		(start 107.45852 120.75)
+		(end 105.251 122.95752)
 		(width 0.3)
 		(layer "F.Cu")
@@
 	)
 	(segment
-		(start 104.625 125.875)
-		(end 105.75 124.75)
-		(width 0.3)
-		(layer "F.Cu")
-		(net 118)
-	)
-	(segment
 		(start 108.545 120.75)
 		(end 109.5 120.75)
@@
 	)
 	(segment
+		(start 108.545 120.75)
+		(end 107.45852 120.75)
+		(width 0.3)
+		(layer "F.Cu")
+		(net 118)
+	)
+	(segment
 		(start 107.5 120.25)
 		(end 108.545 120.25)
@@
 	)
 	(segment
-		(start 105.249 124.499)
-		(end 105.25 124.5)
-		(width 0.3)
-		(layer "F.Cu")
-		(net 119)
-	)
-	(segment
-		(start 105.249 122.251)
-		(end 105.249 124.499)
-		(width 0.3)
-		(layer "F.Cu")
-		(net 119)
-	)
-	(segment
-		(start 107.25 120.25)
-		(end 105.249 122.251)
-		(width 0.3)
-		(layer "F.Cu")
-		(net 119)
-	)
-	(segment
 		(start 107.5 119.25)
 		(end 107.25 119.5)
@@
 	)
 	(segment
-		(start 103.75 126)
-		(end 103.75 126.43)
-		(width 0.3)
-		(layer "F.Cu")
-		(net 119)
-	)
-	(segment
 		(start 107.25 119.5)
 		(end 107.25 120)
@@
 	)
 	(segment
-		(start 105.25 124.5)
-		(end 103.75 126)
+		(start 103.75 126.43)
+		(end 103.75 125.523496)
+		(width 0.3)
+		(layer "F.Cu")
+		(net 119)
+	)
+	(segment
+		(start 103.75 125.523496)
+		(end 104.75 124.523496)
+		(width 0.3)
+		(layer "F.Cu")
+		(net 119)
+	)
+	(segment
+		(start 104.75 124.523496)
+		(end 104.75 122.75)
 		(width 0.3)
 		(layer "F.Cu")
@@
 	)
 	(segment
-		(start 107.5 120.25)
+		(start 107.25 120.25)
+		(end 107.5 120.25)
+		(width 0.3)
+		(layer "F.Cu")
+		(net 119)
+	)
+	(segment
+		(start 104.75 122.75)
 		(end 107.25 120.25)
 		(width 0.3)
