File: MouseWB5/MouseWB5.kicad_pcb (KiCad board)
At the start: 6 copper layers, 65.5 x 40 mm, 67 parts, among them J1 USB_C_Receptacle_USB2.0_14P, J10 Conn_01x09_Socket, J11 TC2030, J2 Conn_01x11_Socket, J3 Conn_01x09_Socket, J9 Conn_01x02_Socket, M1 Conn_01x02_Socket, M2 Conn_01x02_Socket, M3 Conn_01x02_Socket, M4 Conn_01x02_Socket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

Commit message: work
Routing:
- net GND: track 65.6 -> 69.9 mm
Changed lines of the file:
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@@
 			(outputformat 1)
 			(mirror no)
-			(drillshape 1)
+			(drillshape 0)
 			(scaleselection 1)
-			(outputdirectory "")
+			(outputdirectory "production/")
 		)
 	)
@@
 	)
 	(segment
+		(start 104.55 100.8)
+		(end 104.699 100.651)
+		(width 0.3)
+		(layer "F.Cu")
+		(net 80)
+	)
+	(segment
 		(start 131.25 100.75)
 		(end 131.8 100.75)
@@
 	)
 	(segment
+		(start 104.699 100.651)
+		(end 108.7 100.651)
+		(width 0.3)
+		(layer "F.Cu")
+		(net 80)
+	)
+	(segment
 		(start 101.0751 103.5751)
 		(end 101 103.5)
@@
 		(min_thickness 0.25)
 		(filled_areas_thickness no)
-		(fill yes
+		(fill
 			(thermal_gap 0.5)
 			(thermal_bridge_width 0.5)
@@
 		(min_thickness 0.25)
 		(filled_areas_thickness no)
-		(fill yes
+		(fill
 			(thermal_gap 0.5)
 			(thermal_bridge_width 0.5)
@@
 		(min_thickness 0.25)
 		(filled_areas_thickness no)
-		(fill yes
+		(fill
 			(thermal_gap 0.5)
 			(thermal_bridge_width 0.5)

Commit message: work
Routing:
- net GND: track 69.9 -> 75.3 mm, vias 46 -> 45
Changed lines of the file:
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@@
+	)
+	(segment
+		(start 112.75 119.597599)
+		(end 113.4512 120.2988)
+		(width 0.3)
+		(layer "F.Cu")
+		(net 80)
 	)
 	(segment
@@
 	)
 	(segment
+		(start 136.25 139)
+		(end 134.95 139)
+		(width 0.5)
+		(layer "F.Cu")
+		(net 80)
+	)
+	(segment
 		(start 131.8 100.75)
 		(end 132.55 101.5)
@@
 	)
 	(segment
+		(start 112.76 115)
+		(end 112.76 119.607599)
+		(width 0.5)
+		(layer "F.Cu")
+		(net 80)
+	)
+	(segment
 		(start 118 122)
 		(end 118 121.25)
@@
 	)
 	(segment
-		(start 112.5 118.5)
-		(end 112.76 118.24)
-		(width 0.3)
-		(layer "F.Cu")
-		(net 80)
-	)
-	(segment
 		(start 101.0751 110.3251)
 		(end 101 110.25)
@@
 	)
 	(segment
-		(start 112.76 115.75)
-		(end 112.76 117.5)
-		(width 0.3)
-		(layer "F.Cu")
-		(net 80)
-	)
-	(segment
-		(start 112.3 118.5)
-		(end 112.75 118.95)
-		(width 0.3)
+		(start 106.65 113.45)
+		(end 104.75 111.55)
+		(width 0.5)
 		(layer "F.Cu")
 		(net 80)
@@
 		(end 107.63 115.68)
 		(width 0.5)
-		(layer "F.Cu")
-		(net 80)
-	)
-	(segment
-		(start 112.75 119.597599)
-		(end 113.4512 120.2988)
-		(width 0.3)
 		(layer "F.Cu")
 		(net 80)
@@
 	)
 	(segment
-		(start 112.76 115)
-		(end 112.76 115.75)
-		(width 0.3)
-		(layer "F.Cu")
-		(net 80)
-	)
-	(segment
 		(start 158.235 102.75)
 		(end 159.25 102.75)
@@
 	)
 	(segment
-		(start 104.75 110.799)
-		(end 104.7 110.749)
+		(start 109.25 113.45)
+		(end 113.75 113.45)
 		(width 0.5)
 		(layer "F.Cu")
@@
 		(end 103.625 138.535)
 		(width 0.5)
-		(layer "F.Cu")
-		(net 80)
-	)
-	(segment
-		(start 135.75 138.5)
-		(end 134.45 138.5)
-		(width 0.5)
-		(layer "F.Cu")
-		(net 80)
-	)
-	(segment
-		(start 112.76 118.24)
-		(end 112.76 115.75)
-		(width 0.3)
 		(layer "F.Cu")
 		(net 80)
@@
 	)
 	(segment
-		(start 104.75 111.55)
-		(end 104.75 110.799)
+		(start 107 113.45)
+		(end 106.65 113.45)
+		(width 0.5)
+		(layer "F.Cu")
+		(net 80)
+	)
+	(segment
+		(start 112.76 119.607599)
+		(end 113.4524 120.299999)
 		(width 0.5)
 		(layer "F.Cu")
@@
 	)
 	(segment
-		(start 112.3 118.5)
-		(end 112.5 118.5)
-		(width 0.3)
-		(layer "F.Cu")
-		(net 80)
-	)
-	(segment
 		(start 155.349999 115.4)
 		(end 154.5 115.4)
@@
 	)
 	(segment
+		(start 134.95 139)
+		(end 134.45 138.5)
+		(width 0.5)
+		(layer "F.Cu")
+		(net 80)
+	)
+	(segment
 		(start 128.27 107.25)
 		(end 128.27 106.48)
@@
 	)
 	(segment
-		(start 136.25 139)
-		(end 135.75 138.5)
-		(width 0.5)
-		(layer "F.Cu")
-		(net 80)
-	)
-	(segment
-		(start 112.75 118.95)
-		(end 112.75 119.597599)
-		(width 0.3)
-		(layer "F.Cu")
-		(net 80)
-	)
-	(segment
 		(start 154.4 115.5)
 		(end 154.5 115.4)
@@
 	)
 	(via
-		(at 104.7 110.749)
-		(size 0.6)
-		(drill 0.3)
-		(layers "F.Cu" "B.Cu")
-		(net 80)
-	)
-	(via
 		(at 137.25 139)
 		(size 0.6)
@@
 	)
 	(via
-		(at 112.3 118.5)
-		(size 0.6)
-		(drill 0.3)
+		(at 112.75 118.5)
+		(size 0.6)
+		(drill 0.3)

Commit message: work
Parts:
- renumbered J11 to DBG1
Routing:
- net GND: track 75.3 -> 79.0 mm, vias 45 -> 44
- net /SWDIO: track 0.69 -> 3.29 mm, vias 1 -> 2
- net /SWO: track 0.69 -> 3.19 mm, vias 1 -> 2
- net /SWCLK: track 0.68 -> 3.14 mm, vias 1 -> 2
- net /RST: track 0.75 -> 2.10 mm, vias 1 -> 2
- net +3V3: vias 1 -> 0
Changed lines of the file:
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@@
 			(layer "F.Fab")
 		)
-		(fp_text user "${REFERENCE}"
-			(at 0 0 90)
-			(layer "F.Fab")
-			(effects
-				(font
-					(size 0.5 0.5)
-					(thickness 0.08)
-				)
-			)
-		)
 		(pad "1" smd roundrect
 			(at -0.95 0 270)
@@
 		(descr "Tag-Connect programming header; http://www.tag-connect.com/Materials/TC2030-IDC-NL.pdf")
 		(tags "tag connect programming header pogo pins")
-		(property "Reference" "J11"
+		(property "Reference" "DBG1"
 			(at 0 2.7 0)
 			(layer "F.SilkS")
@@
 			(layer "F.CrtYd")
 		)
-		(fp_text user "KEEPOUT"
-			(at 0 0 0)
-			(layer "Cmts.User")
-			(effects
-				(font
-					(size 0.4 0.4)
-					(thickness 0.07)
-				)
-			)
-		)
-		(fp_text user "${REFERENCE}"
-			(at 0 0 0)
-			(layer "F.Fab")
-			(effects
-				(font
-					(size 1 1)
-					(thickness 0.15)
-				)
-			)
-		)
 		(pad "" np_thru_hole circle
 			(at -2.54 0 180)
@@
 			(layer "F.Fab")
 		)
-		(fp_text user "${REFERENCE}"
-			(at 0 0 90)
-			(layer "F.Fab")
-			(effects
-				(font
-					(size 0.5 0.5)
-					(thickness 0.08)
-				)
-			)
-		)
 		(pad "1" smd roundrect
 			(at -0.95 0 270)
@@
 	)
 	(segment
-		(start 105.75 123.25)
-		(end 106.786 122.214)
+		(start 104.875 127.725)
+		(end 105.25 127.35)
 		(width 0.2)
 		(layer "F.Cu")
@@
 	)
 	(segment
-		(start 108.309 122.214)
-		(end 108.545 122.45)
-		(width 0.2)
-		(layer "F.Cu")
-		(net 79)
-	)
-	(segment
-		(start 105.75 125)
-		(end 105.75 123.25)
+		(start 105.25 125.5)
+		(end 105.75 125)
 		(width 0.2)
 		(layer "F.Cu")
@@
 	)
 	(segment
-		(start 107 114.552832)
-		(end 106.052832 114.552832)
-		(width 0.5)
+		(start 106.786 122.214)
+		(end 108.309 122.214)
+		(width 0.2)
 		(layer "F.Cu")
 		(net 79)
 	)
 	(segment
-		(start 104.875 128.325)
-		(end 104.875 127.875)
+		(start 105.25 127.35)
+		(end 105.25 125.5)
+		(width 0.2)
+		(layer "F.Cu")
+		(net 79)
+	)
+	(segment
+		(start 105.75 125)
+		(end 105.75 123.25)
 		(width 0.2)
 		(layer "F.Cu")
@@
 	)
 	(segment
+		(start 107 114.552832)
+		(end 106.052832 114.552832)
+		(width 0.5)
+		(layer "F.Cu")
+		(net 79)
+	)
+	(segment
 		(start 104.95 113.45)
 		(end 104.75 113.45)
@@
 	)
 	(segment
-		(start 105.25 125.5)
-		(end 105.75 125)
+		(start 105.75 123.25)
+		(end 106.786 122.214)
 		(width 0.2)
 		(layer "F.Cu")
@@
 	)
 	(segment
-		(start 105.25 127.5)
-		(end 105.25 125.5)
+		(start 108.309 122.214)
+		(end 108.545 122.45)
 		(width 0.2)
 		(layer "F.Cu")
@@
 	)
 	(segment
-		(start 104.875 127.875)
-		(end 105.25 127.5)
-		(width 0.2)
-		(layer "F.Cu")
-		(net 79)
-	)
-	(segment
-		(start 106.786 122.214)
-		(end 108.309 122.214)
-		(width 0.2)
-		(layer "F.Cu")
-		(net 79)
-	)
-	(segment
 		(start 108.545 117.55)
 		(end 109.5446 117.55)
@@
 		(net 79)
 	)
+	(segment
+		(start 104.875 128.325)
+		(end 104.875 127.725)
+		(width 0.2)
+		(layer "F.Cu")
+		(net 79)
+	)
 	(via
 		(at 107 114.552832)
@@
 	)
 	(segment
-		(start 103.5 128.325)
-		(end 103.5 127.75)
-		(width 0.2)
-		(layer "F.Cu")
-		(net 80)
-	)
-	(segment
 		(start 136.25 139)
 		(end 134.95 139)
@@
 	)
 	(segment
-		(start 103.5 127.75)
-		(end 103.375 127.75)
-		(width 0.2)
-		(layer "F.Cu")
-		(net 80)
-	)
-	(segment
 		(start 111.725 123.9)
 		(end 112.6125 123.9)
@@
 	)
 	(segment
+		(start 103.667843 124.967843)
+		(end 103.667843 124.537843)
+		(width 0.2)
+		(layer "F.Cu")
+		(net 80)
+	)
+	(segment
+		(start 103.5 127.61987)
+		(end 103.2 127.31987)
+		(width 0.2)
+		(layer "F.Cu")
+		(net 80)
+	)
+	(segment
 		(start 131.25 100.75)
 		(end 131.8 100.75)
@@
 	)
 	(segment
+		(start 103.2 127.31987)
+		(end 103.2 125.435686)
+		(width 0.2)
+		(layer "F.Cu")
+		(net 80)
+	)
+	(segment
 		(start 107 113.45)
 		(end 107.751 114.201)
@@
 	)
 	(segment
+		(start 103.2 125.435686)
+		(end 103.667843 124.967843)
+		(width 0.2)
+		(layer "F.Cu")
+		(net 80)
+	)
+	(segment
 		(start 101.0751 134.5751)
 		(end 101.0751 133.3251)
@@
 	)
 	(segment
+		(start 103.5 128.325)
+		(end 103.5 127.61987)
+		(width 0.2)
+		(layer "F.Cu")
+		(net 80)
+	)
+	(segment
 		(start 138.73 133.27)
 		(end 138.73 132.75)
@@
 	)
 	(segment
+		(start 103.667843 124.537843)
+		(end 103.45 124.32)
+		(width 0.2)
+		(layer "F.Cu")
+		(net 80)
+	)
+	(segment
 		(start 154.4 115.5)
 		(end 154.5 115.4)
@@
 	)
 	(via
-		(at 103.375 127.75)
-		(size 0.6)
-		(drill 0.3)
-		(layers "F.Cu" "B.Cu")
-		(net 80)
-	)
-	(via
 		(at 105.25 101.5)
 		(size 0.6)
@@
 		(net 81)
 	)
-	(via
-		(at 102.8 128.306215)
-		(size 0.6)
-		(drill 0.3)
-		(layers "F.Cu" "B.Cu")
-		(net 81)
-	)
 	(segment
 		(start 163.376 122.72504)
@@
 	)
 	(segment
+		(start 105.775 125.975)
+		(end 105.775 128.325)
+		(width 0.2)
+		(layer "F.Cu")
+		(net 100)
+	)
+	(segment
 		(start 106.5 103.52)
 		(end 106.5 104.2)
@@
 		(net 100)
 	)
+	(segment
+		(start 105.85 125.9)
+		(end 105.775 125.975)
+		(width 0.2)
+		(layer "F.Cu")
+		(net 100)
+	)
+	(via
+		(at 105.85 125.9)
+		(size 0.6)
+		(drill 0.3)
+		(layers "F.Cu" "B.Cu")
+		(net 100)
+	)
 	(via
 		(at 106.5 104.2)
@@
 	)
 	(segment
+		(start 108.025 126.075)
+		(end 108.2 125.9)
+		(width 0.2)
+		(layer "F.Cu")
+		(net 101)
+	)
+	(segment
 		(start 105.23 104.18)
 		(end 105.25 104.2)
@@
 		(net 101)
 	)
+	(segment
+		(start 108.025 128.325)
+		(end 108.025 126.075)
+		(width 0.2)
+		(layer "F.Cu")
+		(net 101)
+	)
 	(via
 		(at 105.25 104.2)
@@
 		(net 101)
 	)
+	(via
+		(at 108.2 125.9)
+		(size 0.6)
+		(drill 0.3)
+		(layers "F.Cu" "B.Cu")
+		(net 101)
+	)
+	(segment
+		(start 109.85 131.5)
+		(end 111.2 131.5)
+		(width 0.2)
+		(layer "F.Cu")
+		(net 102)
+	)
 	(segment
 		(start 106.5 102.25)
@@
 	)
 	(via
+		(at 111.2 131.5)
+		(size 0.6)
+		(drill 0.3)
+		(layers "F.Cu" "B.Cu")
+		(net 102)
+	)
+	(via
 		(at 106.5 101.5)
 		(size 0.6)
@@
 	)
 	(segment
+		(start 106.225 126.375)
+		(end 106.650003 125.949997)
+		(width 0.2)
+		(layer "F.Cu")
+		(net 103)
+	)
+	(segment
+		(start 106.650003 125.949997)
+		(end 106.650003 125.9)
+		(width 0.2)
+		(layer "F.Cu")
+		(net 103)
+	)
+	(segment
 		(start 107.77 103.52)
 		(end 107.77 104.18)
@@
 	)
 	(segment
+		(start 106.225 128.325)
+		(end 106.225 126.375)
+		(width 0.2)
+		(layer "F.Cu")
+		(net 103)
+	)
+	(segment
 		(start 107.77 104.18)
 		(end 107.75 104.2)
@@
 		(size 0.6)
 		(drill 0.3)
+		(layers "F.Cu" "B.Cu")
+		(net 103)
+	)
+	(via
+		(at 106.650003 125.9)
+		(size 0.6)
+		(drill 0.3)

Commit message: work
Parts:
- removed Q1: FDN327N, FDN327N:SSOT-3
- added D3: BAT54J, Diode_SMD:D_SOD-323F, F.Cu at (153.2, 122.8)
- added Q2: CSD13380F3, Package_DFN_QFN:Texas_PicoStar_DFN-3_0.69x0.60mm, F.Cu at (151.5, 122.8)
- added R9: 20k, Resistor_SMD:R_0402_1005Metric, F.Cu at (151.5, 121.0)
Connections:
- J1 pad A5: Net-(J1-CC1) -> unconnected-(J1-CC1-PadA5)
- M5 pad 1: unconnected-(M5-Pin_1-Pad1) -> +BATT
- M5 pad 2: unconnected-(M5-Pin_2-Pad2) -> Net-(D3-A)
- R1 pad 1: GND -> unconnected-(R1-Pad1)
- R1 pad 2: Net-(J1-CC1) -> unconnected-(R1-Pad2)
Routing:
- net +BATT: track 205.2 -> 211.8 mm
- net Net-(J1-CC1): track 5.67 -> 0.00 mm
- net (no net): track 0.00 -> 5.67 mm
- net Net-(D3-A): track 0.00 -> 4.99 mm
- net GND: track 79.0 -> 83.4 mm, vias 44 -> 47
- net /FAN_CTRL: track 0.00 -> 1.04 mm
Other:
- board text removed: "NMOS"

Commit message: work
Routing:
- net /FAN_CTRL: track 1.04 -> 40.1 mm
- net +1V8: track 154.0 -> 157.0 mm
- net GND: vias 47 -> 48
Changed lines of the file:
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@@
+	)
+	(via
+		(at 123.75 120)
+		(size 0.6)
+		(drill 0.3)
+		(layers "F.Cu" "B.Cu")
+		(free yes)
+		(net 80)
 	)
 	(via
@@
 	)
 	(segment
-		(start 130.25 109.451)
-		(end 130.25 110)
-		(width 0.5)
-		(layer "F.Cu")
-		(net 137)
-	)
-	(segment
 		(start 161.292893 111.042893)
 		(end 160.884786 111.451)
@@
 	)
 	(segment
+		(start 130.25 109.451)
+		(end 130.25 111.5)
+		(width 0.5)
+		(layer "F.Cu")
+		(net 137)
+	)
+	(segment
 		(start 121.25 118.5)
 		(end 121 118.25)
@@
 	)
 	(via
-		(at 130.25 110)
+		(at 130.25 111.5)
 		(size 0.6)
 		(drill 0.3)
@@
 	)
 	(segment
+		(start 130.25 105.25)
+		(end 130.41538 105.08462)
+		(width 0.5)
+		(layer "B.Cu")
+		(net 137)
+	)
+	(segment
+		(start 130.25 111.5)
+		(end 130.25 105.25)
+		(width 0.5)
+		(layer "B.Cu")
+		(net 137)
+	)
+	(segment
 		(start 115.356037 124.55)
 		(end 114.635037 125.271)
@@
 	)
 	(segment
-		(start 130.25 110)
-		(end 130.25 105.25)
-		(width 0.5)
-		(layer "B.Cu")
-		(net 137)
-	)
-	(segment
 		(start 114.635037 125.271)
 		(end 111.021 125.271)
@@
 	)
 	(segment
-		(start 130.25 105.25)
-		(end 130.41538 105.08462)
-		(width 0.5)
-		(layer "B.Cu")
-		(net 137)
+		(start 136.349 128.651)
+		(end 128.901 128.651)
+		(width 0.3)
+		(layer "F.Cu")
+		(net 162)
+	)
+	(segment
+		(start 122.423166 123.25)
+		(end 119.211583 126.461583)
+		(width 0.3)
+		(layer "F.Cu")
+		(net 162)
 	)
 	(segment
@@
 	)
 	(segment
+		(start 151.5 121.5)
+		(end 151.25 121.25)
+		(width 0.3)
+		(layer "F.Cu")
+		(net 162)
+	)
+	(segment
 		(start 151.274 121.976)
 		(end 151.274 122.449)
@@
 	)
 	(segment
+		(start 151.25 121.25)
+		(end 143.75 121.25)
+		(width 0.3)
+		(layer "F.Cu")
+		(net 162)
+	)
+	(segment
+		(start 123.5 123.25)
+		(end 122.423166 123.25)
+		(width 0.3)
+		(layer "F.Cu")
+		(net 162)
+	)
+	(segment
+		(start 128.901 128.651)
+		(end 123.5 123.25)
+		(width 0.3)
+		(layer "F.Cu")
+		(net 162)
+	)
+	(segment
 		(start 151.5 121.75)
 		(end 151.274 121.976)
 		(width 0.3)
 		(layer "F.Cu")
+		(net 162)
+	)
+	(segment
+		(start 143.75 121.25)
+		(end 136.349 128.651)
+		(width 0.3)
+		(layer "F.Cu")

Commit message: work
Parts:
- U5: value LSM6DSO -> LSM6DS0
Connections:
- U1 pad 28: VBUS -> unconnected-(U1-PA10-Pad28)
- U1 pad 7: unconnected-(U1-PC3-Pad7) -> /FAN_CTRL
Routing:
- net VBUS: track 29.2 -> 20.4 mm
- net /FAN_CTRL: track 40.1 -> 47.5 mm
- net unconnected-(U1-PC2-Pad8): track 0.00 -> 5.65 mm
- net unconnected-(U1-PC1-Pad9): track 0.00 -> 5.02 mm

Commit message: work
Routing:
- net /IMU_INT1: track 9.38 -> 2.12 mm, vias 0 -> 1
- net /IMU_MISO: track 6.84 -> 2.35 mm, vias 0 -> 1
- net /IMU_MOSI: track 6.39 -> 3.19 mm, vias 0 -> 1
- net /IMU_CLK: track 6.18 -> 3.75 mm, vias 0 -> 1
- net /IMU_CS: track 5.74 -> 4.64 mm, vias 0 -> 1
- net /IMU_INT2: track 7.47 -> 7.67 mm, vias 0 -> 1
- net GND: vias 48 -> 49
Changed lines of the file:
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@@
 	)
 	(segment
-		(start 120.25 120.9125)
-		(end 120.25 122)
-		(width 0.25)
+		(start 123.428 122.028)
+		(end 120.918801 122.028)
+		(width 0.2)
 		(layer "F.Cu")
 		(net 56)
 	)
 	(segment
-		(start 120.25 122.181095)
-		(end 117.090547 125.340547)
-		(width 0.25)
+		(start 123.95 122.55)
+		(end 123.428 122.028)
+		(width 0.2)
 		(layer "F.Cu")
 		(net 56)
 	)
 	(segment
-		(start 120.25 122)
-		(end 120.25 122.181095)
-		(width 0.25)
+		(start 120.918801 122.028)
+		(end 120.25 121.359199)
+		(width 0.2)
 		(layer "F.Cu")
 		(net 56)
 	)
 	(segment
-		(start 117.090547 125.340548)
-		(end 117.090547 125.340547)
-		(width 0.25)
+		(start 120.25 121.359199)
+		(end 120.25 120.9125)
+		(width 0.2)
 		(layer "F.Cu")
 		(net 56)
 	)
+	(via
+		(at 123.95 122.55)
+		(size 0.6)
+		(drill 0.3)
+		(layers "F.Cu" "B.Cu")
+		(net 56)
+	)
 	(segment
 		(start 112.45 132.05)
@@
 	)
 	(via
-		(at 123.75 120)
+		(at 121.05 114.45)
 		(size 0.6)
 		(drill 0.3)
@@
 	)
 	(via
+		(at 123 119.9)
+		(size 0.6)
+		(drill 0.3)
+		(layers "F.Cu" "B.Cu")
+		(free yes)
+		(net 79)
+	)
+	(via
 		(at 101 110.25)
 		(size 0.6)
@@
 	)
 	(segment
-		(start 120.75 122.318905)
-		(end 117.375 125.693905)
-		(width 0.25)
+		(start 123.95 121.7)
+		(end 123.877 121.627)
+		(width 0.2)
 		(layer "F.Cu")
 		(net 86)
 	)
 	(segment
-		(start 120.75 120.9125)
-		(end 120.75 122.318905)
-		(width 0.25)
+		(start 120.75 121.292099)
+		(end 120.75 120.9125)
+		(width 0.2)
 		(layer "F.Cu")
 		(net 86)
 	)
 	(segment
-		(start 121.9125 122.44969)
-		(end 118.280475 126.081715)
-		(width 0.25)
+		(start 123.877 121.627)
+		(end 121.084901 121.627)
+		(width 0.2)
 		(layer "F.Cu")
-		(net 87)
+		(net 86)
+	)
+	(segment
+		(start 121.084901 121.627)
+		(end 120.75 121.292099)
+		(width 0.2)
+		(layer "F.Cu")
+		(net 86)
+	)
+	(via
+		(at 123.95 121.7)
+		(size 0.6)
+		(drill 0.3)
+		(layers "F.Cu" "B.Cu")
+		(net 86)
 	)
 	(segment
 		(start 121.9125 120.75)
-		(end 121.9125 122.44969)
-		(width 0.25)
+		(end 123.150058 120.75)
+		(width 0.2)
+		(layer "F.Cu")
+		(net 87)
+	)
+	(segment
+		(start 123.900059 120)
+		(end 123.949997 120)
+		(width 0.2)
+		(layer "F.Cu")
+		(net 87)
+	)
+	(segment
+		(start 123.150058 120.75)
+		(end 123.900059 120)
+		(width 0.2)
 		(layer "F.Cu")
 		(net 87)
 	)
+	(via
+		(at 123.949997 120)
+		(size 0.6)
+		(drill 0.3)
+		(layers "F.Cu" "B.Cu")
+		(net 87)
+	)
 	(segment
 		(start 135.58076 104.25)
@@
 	)
 	(segment
-		(start 119 119.75)
-		(end 118.886 119.864)
-		(width 0.25)
+		(start 120.752701 122.429)
+		(end 119.562125 121.238424)
+		(width 0.2)
 		(layer "F.Cu")
 		(net 96)
 	)
 	(segment
-		(start 118.886 120.75)
-		(end 118.886 121)
-		(width 0.25)
+		(start 119.211576 121.238424)
+		(end 118.974 121.000848)
+		(width 0.2)
 		(layer "F.Cu")
 		(net 96)
 	)
 	(segment
-		(start 118.886 119.864)
-		(end 118.886 120.75)
-		(width 0.25)
+		(start 123.90006 123.350003)
+		(end 122.979057 122.429)
+		(width 0.2)
 		(layer "F.Cu")
 		(net 96)
 	)
 	(segment
-		(start 119.5875 119.75)
-		(end 119 119.75)
-		(width 0.25)
+		(start 119.223152 119.75)
+		(end 119.5875 119.75)
+		(width 0.2)
 		(layer "F.Cu")
 		(net 96)
 	)
 	(segment
-		(start 118.886 121)
-		(end 119.5 121.614)
-		(width 0.25)
+		(start 118.974 121.000848)
+		(end 118.974 119.999152)
+		(width 0.2)
 		(layer "F.Cu")
 		(net 96)
 	)
 	(segment
-		(start 119.5 121.614)
-		(end 119.5 122.293285)
-		(width 0.25)
+		(start 119.562125 121.238424)
+		(end 119.211576 121.238424)
+		(width 0.2)
 		(layer "F.Cu")
 		(net 96)
 	)
 	(segment
-		(start 119.5 122.293285)
-		(end 118.886 122.907285)
-		(width 0.25)
+		(start 123.95 123.350003)
+		(end 123.90006 123.350003)
+		(width 0.2)
 		(layer "F.Cu")
 		(net 96)
 	)
 	(segment
-		(start 118.886 122.907285)
-		(end 116.646642 125.146642)
-		(width 0.25)
+		(start 118.974 119.999152)
+		(end 119.223152 119.75)
+		(width 0.2)
 		(layer "F.Cu")
 		(net 96)
 	)
 	(segment
-		(start 121.25 122.47438)
-		(end 117.83657 125.88781)
-		(width 0.25)
+		(start 122.979057 122.429)
+		(end 120.752701 122.429)
+		(width 0.2)
+		(layer "F.Cu")
+		(net 96)
+	)
+	(via
+		(at 123.95 123.350003)
+		(size 0.6)
+		(drill 0.3)
+		(layers "F.Cu" "B.Cu")
+		(net 96)
+	)
+	(segment
+		(start 121.25 121.224999)
+		(end 121.25 120.9125)
+		(width 0.2)
 		(layer "F.Cu")
 		(net 97)
 	)
 	(segment
-		(start 121.25 120.9125)
-		(end 121.25 122.47438)
-		(width 0.25)
+		(start 121.251001 121.226)
+		(end 121.25 121.224999)
+		(width 0.2)
+		(layer "F.Cu")
+		(net 97)
+	)
+	(segment
+		(start 123.95 120.800002)
+		(end 123.524002 121.226)
+		(width 0.2)
 		(layer "F.Cu")
 		(net 97)
 	)
 	(segment
+		(start 123.524002 121.226)
+		(end 121.251001 121.226)
+		(width 0.2)
+		(layer "F.Cu")
+		(net 97)
+	)
+	(via
+		(at 123.95 120.800002)
+		(size 0.6)
+		(drill 0.3)
+		(layers "F.Cu" "B.Cu")
+		(net 97)
+	)
+	(segment
 		(start 105.775 125.975)
 		(end 105.775 128.325)
@@
 	)
 	(segment
-		(start 122.75 122.25)
-		(end 118.72438 126.27562)
+		(start 123.95 119.2)
+		(end 121.9625 119.2)
 		(width 0.25)
 		(layer "F.Cu")
@@
 	)
 	(segment
-		(start 122.75 119.5)
-		(end 122.75 122.25)
+		(start 121.9625 119.2)
+		(end 121.9125 119.25)
 		(width 0.25)
 		(layer "F.Cu")
@@
 	)
 	(segment
-		(start 122.5 119.25)
-		(end 122.75 119.5)
+		(start 123.95 119.22698)
+		(end 123.92698 119.25)
 		(width 0.25)
 		(layer "F.Cu")
@@
 	)
 	(segment
-		(start 121.9125 119.25)
-		(end 122.5 119.25)
+		(start 123.95 119.2)
+		(end 123.95 119.22698)
 		(width 0.25)
 		(layer "F.Cu")
 		(net 105)
 	)
+	(via
+		(at 123.95 119.2)
+		(size 0.6)
+		(drill 0.3)
+		(layers "F.Cu" "B.Cu")
+		(net 105)
+	)
 	(segment
 		(start 132.0125 104.75)
@@
 		(min_thickness 0.25)
 		(filled_areas_thickness no)
-		(fill
+		(fill yes
 			(thermal_gap 0.5)
 			(thermal_bridge_width 0.5)
@@
 		(min_thickness 0.25)
 		(filled_areas_thickness no)
-		(fill
+		(fill yes
 			(thermal_gap 0.5)
 			(thermal_bridge_width 0.5)
@@
 		(min_thickness 0.25)
 		(filled_areas_thickness no)
-		(fill
+		(fill yes
 			(thermal_gap 0.5)
 			(thermal_bridge_width 0.5)

Commit message: work
Routing:
- net +1V8: track 157.0 -> 194.9 mm, vias 5 -> 6
- net GND: track 83.4 -> 89.2 mm, vias 49 -> 53
- net unconnected-(U1-PC2-Pad8): track 5.65 -> 0.00 mm
- net unconnected-(U1-PC1-Pad9): track 5.02 -> 0.00 mm
