File: MouseWB5/MouseWB5.kicad_sch (KiCad schematic)
At the start: 68 parts, among them J1 USB_C_Receptacle_USB2.0_14P, J10 Conn_01x09_Socket, J2 Conn_01x11_Socket, J3 Conn_01x09_Socket, J4 Conn_01x02_Socket, J5 Conn_01x02_Socket, J6 Conn_01x02_Socket, J7 Conn_01x02_Socket, J8 Conn_01x02_Socket, J9 Conn_01x02_Socket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

Commit message: work
Parts:
- added U10, U8, U9: TXS0108EPW, TXS0108ERGYR:IC_TXS0108ERGYR, symbol Logic_LevelTranslator:TXS0108EPW
Connections:
- net GND: now also U10.11 (GND), U8.11 (GND), U9.11 (GND)

Commit message: work
Parts:
- U10, U8, U9: footprint TXS0108ERGYR:IC_TXS0108ERGYR -> TXS0108ERGYRslim:VQFN20_RKS_TEX
Changed lines of the file:
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@@
 			)
 		)
-		(property "Footprint" "TXS0108ERGYR:IC_TXS0108ERGYR"
+		(property "Footprint" "TXS0108ERGYRslim:VQFN20_RKS_TEX"
 			(at 394.97 217.17 0)
 			(effects
@@
 			)
 		)
-		(property "Footprint" "TXS0108ERGYR:IC_TXS0108ERGYR"
+		(property "Footprint" "TXS0108ERGYRslim:VQFN20_RKS_TEX"
 			(at 394.97 119.38 0)
 			(effects
@@
 			)
 		)
-		(property "Footprint" "TXS0108ERGYR:IC_TXS0108ERGYR"
+		(property "Footprint" "TXS0108ERGYRslim:VQFN20_RKS_TEX"
 			(at 394.97 165.1 0)
 			(effects

Commit message: work
Parts:
- removed H1, H4: MountingHole, MountingHole:MountingHole_2.1mm, symbol Mechanical:MountingHole
Changed lines of the file:
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@@
-	)
-	(symbol
-		(lib_id "Mechanical:MountingHole")
-		(at 492.76 341.63 0)
-		(unit 1)
-		(exclude_from_sim no)
-		(in_bom no)
-		(on_board yes)
-		(dnp no)
-		(fields_autoplaced yes)
-		(property "Reference" "H4"
-			(at 495.3 340.3599 0)
-			(effects
-				(font
-					(size 1.27 1.27)
-				)
-				(justify left)
-			)
-		)
-		(property "Value" "MountingHole"
-			(at 495.3 342.8999 0)
-			(effects
-				(font
-					(size 1.27 1.27)
-				)
-				(justify left)
-			)
-		)
-		(property "Footprint" "MountingHole:MountingHole_2.1mm"
-			(at 492.76 341.63 0)
-			(effects
-				(font
-					(size 1.27 1.27)
-				)
-				(hide yes)
-			)
-		)
-		(property "Datasheet" "~"
-			(at 492.76 341.63 0)
-			(effects
-				(font
-					(size 1.27 1.27)
-				)
-				(hide yes)
-			)
-		)
-		(property "Description" "Mounting Hole without connection"
-			(at 492.76 341.63 0)
-			(effects
-				(font
-					(size 1.27 1.27)
-				)
-				(hide yes)
-			)
-		)
-		(instances
-			(project "MouseWB5"
-				(path "/3003f723-e5bb-4cdb-ac11-d8017cbd2609"
-					(reference "H4")
-					(unit 1)
-				)
-			)
-		)
 	)
 	(symbol
@@
 					(unit 1)
 				)
-			)
-		)
-	)
-	(symbol
-		(lib_id "Mechanical:MountingHole")
-		(at 492.76 326.39 0)
-		(unit 1)
-		(exclude_from_sim no)
-		(in_bom no)
-		(on_board yes)
-		(dnp no)
-		(fields_autoplaced yes)
-		(property "Reference" "H1"
-			(at 495.3 325.1199 0)
-			(effects
-				(font
-					(size 1.27 1.27)
-				)
-				(justify left)
-			)
-		)
-		(property "Value" "MountingHole"
-			(at 495.3 327.6599 0)
-			(effects
-				(font
-					(size 1.27 1.27)
-				)
-				(justify left)
-			)
-		)
-		(property "Footprint" "MountingHole:MountingHole_2.1mm"
-			(at 492.76 326.39 0)
-			(effects
-				(font
-					(size 1.27 1.27)
-				)
-				(hide yes)
-			)
-		)
-		(property "Datasheet" "~"
-			(at 492.76 326.39 0)
-			(effects
-				(font
-					(size 1.27 1.27)
-				)
-				(hide yes)
-			)
-		)
-		(property "Description" "Mounting Hole without connection"
-			(at 492.76 326.39 0)
-			(effects
-				(font
-					(size 1.27 1.27)
-				)
-				(hide yes)
-			)
-		)
-		(instances
-			(project "MouseWB5"
-				(path "/3003f723-e5bb-4cdb-ac11-d8017cbd2609"
-					(reference "H1")
-					(unit 1)
-				)

Commit message: work
Parts:
- removed U7: LP5912-1.8DRV, Package_SON:WSON-6-1EP_2x2mm_P0.65mm_EP1x1.6mm_ThermalVias, symbol Regulator_Linear:LP5912-1.8DRV
- added U7: LP5912-3.3DRV, Package_SON:WSON-6-1EP_2x2mm_P0.65mm_EP1x1.6mm_ThermalVias, symbol Regulator_Linear:LP5912-3.3DRV
Connections:
- net +1V8: now also C5.1, J10.3 (Pin_3), J2.3 (Pin_3), J3.3 (Pin_3), U4.1 (OUT); no longer C10.1, J10.2 (Pin_2), J2.2 (Pin_2), J3.2 (Pin_2)
- net +3V3: now also C10.1, J10.2 (Pin_2), J2.2 (Pin_2), J3.2 (Pin_2), U7.1 (OUT); no longer C5.1, J10.3 (Pin_3), J2.3 (Pin_3), J3.3 (Pin_3), U4.1 (OUT)
- net +BATT: now also U7.4 (EN), U7.6 (IN)
- net GND: now also U7.5 (GND), U7.7 (EP)

Commit message: work
Parts:
- removed DBG1: Conn_01x03_Socket, Connector_JST:JST_SH_SM03B-SRSS-TB_1x03-1MP_P1.00mm_Horizontal, symbol Connector:Conn_01x03_Socket
- added J11: TC2030, Connector:Tag-Connect_TC2030-IDC-NL_2x03_P1.27mm_Vertical, symbol Connector:TC2030
Changed lines of the file:
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@@
 	)
 	(symbol
-		(lib_id "Connector:Conn_01x03_Socket")
-		(at 285.75 218.44 0)
-		(unit 1)
-		(exclude_from_sim no)
-		(in_bom yes)
-		(on_board yes)
-		(dnp no)
-		(fields_autoplaced yes)
-		(property "Reference" "DBG1"
-			(at 287.02 217.1699 0)
-			(effects
-				(font
-					(size 1.27 1.27)
-				)
-				(justify left)
-			)
-		)
-		(property "Value" "Conn_01x03_Socket"
-			(at 287.02 219.7099 0)
-			(effects
-				(font
-					(size 1.27 1.27)
-				)
-				(justify left)
-			)
-		)
-		(property "Footprint" "Connector_JST:JST_SH_SM03B-SRSS-TB_1x03-1MP_P1.00mm_Horizontal"
-			(at 285.75 218.44 0)
-			(effects
-				(font
-					(size 1.27 1.27)
-				)
-				(hide yes)
-			)
-		)
-		(property "Datasheet" "~"
-			(at 285.75 218.44 0)
-			(effects
-				(font
-					(size 1.27 1.27)
-				)
-				(hide yes)
-			)
-		)
-		(property "Description" "Generic connector, single row, 01x03, script generated"
-			(at 285.75 218.44 0)
-			(effects
-				(font
-					(size 1.27 1.27)
-				)
-				(hide yes)
-			)
-		)
-		(pin "3"
-		)
-		(pin "2"
-		)
-		(pin "1"
-		)
-		(instances
-			(project ""
-				(path "/3003f723-e5bb-4cdb-ac11-d8017cbd2609"
-					(reference "DBG1")
-					(unit 1)
-				)
-			)
-		)
-	)
-	(symbol
 		(lib_id "Connector:Conn_01x02_Socket")
 		(at 39.37 175.26 180)
@@
 					(unit 1)
 				)
+			)
+		)
+	)
+	(symbol
+		(lib_id "Connector:TC2030")
+		(at 295.91 218.44 90)
+		(unit 1)
+		(exclude_from_sim no)
+		(in_bom no)
+		(on_board yes)
+		(dnp no)
+		(fields_autoplaced yes)
+		(property "Reference" "J11"
+			(at 304.8 215.8999 90)
+			(effects
+				(font
+					(size 1.27 1.27)
+				)
+				(justify right)
+			)
+		)
+		(property "Value" "TC2030"
+			(at 304.8 218.4399 90)
+			(effects
+				(font
+					(size 1.27 1.27)
+				)
+				(justify right)
+			)
+		)
+		(property "Footprint" "Connector:Tag-Connect_TC2030-IDC-NL_2x03_P1.27mm_Vertical"
+			(at 295.91 217.17 0)
+			(effects
+				(font
+					(size 1.27 1.27)
+				)
+				(hide yes)
+			)
+		)
+		(property "Datasheet" "https://www.tag-connect.com/wp-content/uploads/bsk-pdf-manager/2019/12/TC2030-IDC-NL-Datasheet-Rev-B.pdf"
+			(at 295.91 217.17 0)
+			(effects
+				(font
+					(size 1.27 1.27)
+				)
+				(hide yes)
+			)
+		)
+		(property "Description" "Tag-Connect’s 6-pins connector"
+			(at 295.91 218.44 0)
+			(effects
+				(font
+					(size 1.27 1.27)
+				)
+				(hide yes)
+			)
+		)
+		(pin "4"
+		)
+		(pin "5"
+		)
+		(pin "3"
+		)
+		(pin "1"
+		)
+		(pin "6"
+		)
+		(pin "2"
+		)
+		(instances
+			(project ""
+				(path "/3003f723-e5bb-4cdb-ac11-d8017cbd2609"
+					(reference "J11")
+					(unit 1)
+				)

Commit message: work
Parts:
- removed U10, U8, U9: TXS0108EPW, TXS0108ERGYRslim:VQFN20_RKS_TEX, symbol Logic_LevelTranslator:TXS0108EPW

Commit message: work
Connections:
- net +1V8: now also J11.1
- net GND: now also J11.5
- net RST: now also J11.3
- net SWCLK: now also J11.4
- net SWDIO: now also J11.2
- net SWO: now reaches U1.21 (PB3)
- net SWO: now also J11.6
Changed lines of the file:
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@@
 		)
 	)
-	(text_box "R.PI SWD DEBUG CONNECTOR"
+	(text_box "DEBUG CONNECTOR"
 		(exclude_from_sim no)
-		(at 250.19 198.12 0)
+		(at 262.89 196.85 0)
 		(size 69.85 43.18)
 		(margins 0.9525 0.9525 0.9525 0.9525)
@@
 	(wire
 		(pts
-			(xy 275.59 220.98) (xy 280.67 220.98)
-		)
-		(stroke
-			(width 0)
-			(type default)
-		)
-	)
-	(wire
-		(pts
 			(xy 292.1 293.37) (xy 292.1 295.91)
 		)
@@
 	(wire
 		(pts
-			(xy 309.88 284.48) (xy 309.88 285.75)
+			(xy 185.42 204.47) (xy 193.04 204.47)
 		)
 		(stroke
@@
 	(wire
 		(pts
-			(xy 59.69 243.84) (xy 60.96 243.84)
+			(xy 309.88 284.48) (xy 309.88 285.75)
 		)
 		(stroke
@@
 	(wire
 		(pts
-			(xy 35.56 134.62) (xy 44.45 134.62)
+			(xy 59.69 243.84) (xy 60.96 243.84)
 		)
 		(stroke
@@
 	(wire
 		(pts
-			(xy 72.39 182.88) (xy 80.01 182.88)
+			(xy 35.56 134.62) (xy 44.45 134.62)
 		)
 		(stroke
@@
 	(wire
 		(pts
-			(xy 160.02 153.67) (xy 143.51 153.67)
+			(xy 72.39 182.88) (xy 80.01 182.88)
 		)
 		(stroke
@@
 	(wire
 		(pts
-			(xy 304.8 284.48) (xy 304.8 281.94)
+			(xy 160.02 153.67) (xy 143.51 153.67)
 		)
 		(stroke
@@
 	(wire
 		(pts
-			(xy 275.59 215.9) (xy 280.67 215.9)
+			(xy 304.8 284.48) (xy 304.8 281.94)
 		)
 		(stroke
@@
 	(wire
 		(pts
-			(xy 278.13 218.44) (xy 280.67 218.44)
-		)
-		(stroke
-			(width 0)
-			(type default)
-		)
-	)
-	(wire
-		(pts
 			(xy 292.1 290.83) (xy 311.15 290.83)
 		)
@@
 		)
 	)
+	(label "SWO"
+		(at 298.45 210.82 90)
+		(effects
+			(font
+				(size 1.27 1.27)
+			)
+			(justify left bottom)
+		)
+	)
 	(label "IMU_MISO"
 		(at 34.29 251.46 0)
@@
 		)
 	)
+	(label "SWO"
+		(at 193.04 204.47 180)
+		(effects
+			(font
+				(size 1.27 1.27)
+			)
+			(justify right bottom)
+		)
+	)
 	(label "L_EN"
 		(at 77.47 132.08 0)
@@
 		)
 	)
+	(label "RST"
+		(at 295.91 223.52 270)
+		(effects
+			(font
+				(size 1.27 1.27)
+			)
+			(justify right bottom)
+		)
+	)
+	(label "SWCLK"
+		(at 295.91 210.82 90)
+		(effects
+			(font
+				(size 1.27 1.27)
+			)
+			(justify left bottom)
+		)
+	)
 	(label "IMU_CS"
 		(at 34.29 266.7 0)
@@
 		)
 	)
-	(label "LED_INPUT"
-		(at 31.75 373.38 0)
+	(label "SWDIO"
+		(at 293.37 210.82 90)
 		(effects
 			(font
@@
 		)
 	)
-	(label "SENSE_LR"
-		(at 35.56 134.62 0)
+	(label "LED_INPUT"
+		(at 31.75 373.38 0)
 		(effects
 			(font
@@
 		)
 	)
-	(label "IMU_MOSI"
-		(at 34.29 261.62 0)
+	(label "SENSE_LR"
+		(at 35.56 134.62 0)
 		(effects
 			(font
@@
 		)
 	)
-	(label "SWDIO"
-		(at 275.59 220.98 180)
+	(label "IMU_MOSI"
+		(at 34.29 261.62 0)
 		(effects
 			(font
 				(size 1.27 1.27)
 			)
-			(justify right bottom)
+			(justify left bottom)
 		)
 	)
@@
 		)
 	)
-	(label "SWCLK"
-		(at 275.59 215.9 180)
-		(effects
-			(font
-				(size 1.27 1.27)
-			)
-			(justify right bottom)
-		)
-	)
 	(label "L_PH_B"
 		(at 77.47 124.46 0)
@@
 	)
 	(symbol
-		(lib_id "power:GND")
-		(at 278.13 218.44 270)
-		(unit 1)
-		(exclude_from_sim no)
-		(in_bom yes)
-		(on_board yes)
-		(dnp no)
-		(property "Reference" "#PWR069"
-			(at 271.78 218.44 0)
-			(effects
-				(font
-					(size 1.27 1.27)
-				)
-				(hide yes)
-			)
-		)
-		(property "Value" "GND"
-			(at 275.336 217.424 90)
-			(effects
-				(font
-					(size 1.27 1.27)
-				)
-				(justify right)
-			)
-		)
-		(property "Footprint" ""
-			(at 278.13 218.44 0)
-			(effects
-				(font
-					(size 1.27 1.27)
-				)
-				(hide yes)
-			)
-		)
-		(property "Datasheet" ""
-			(at 278.13 218.44 0)
-			(effects
-				(font
-					(size 1.27 1.27)
-				)
-				(hide yes)
-			)
-		)
-		(property "Description" "Power symbol creates a global label with name \"GND\" , ground"
-			(at 278.13 218.44 0)
-			(effects
-				(font
-					(size 1.27 1.27)
-				)
-				(hide yes)
-			)
-		)
-		(pin "1"
-		)
-		(instances
-			(project "MouseWB5"
-				(path "/3003f723-e5bb-4cdb-ac11-d8017cbd2609"
-					(reference "#PWR069")
-					(unit 1)
-				)
-			)
-		)
-	)
-	(symbol
 		(lib_name "+3V3_1")
 		(lib_id "power:+3V3")
@@
 	(symbol
 		(lib_id "power:GND")
+		(at 298.45 223.52 0)
+		(mirror y)
+		(unit 1)
+		(exclude_from_sim no)
+		(in_bom yes)
+		(on_board yes)
+		(dnp no)
+		(fields_autoplaced yes)
+		(property "Reference" "#PWR0107"
+			(at 298.45 229.87 0)
+			(effects
+				(font
+					(size 1.27 1.27)
+				)
+				(hide yes)
+			)
+		)
+		(property "Value" "GND"
+			(at 298.45 228.6 0)
+			(effects
+				(font
+					(size 1.27 1.27)
+				)
+			)
+		)
+		(property "Footprint" ""
+			(at 298.45 223.52 0)
+			(effects
+				(font
+					(size 1.27 1.27)
+				)
+				(hide yes)
+			)
+		)
+		(property "Datasheet" ""
+			(at 298.45 223.52 0)
+			(effects
+				(font
+					(size 1.27 1.27)
+				)
+				(hide yes)
+			)
+		)
+		(property "Description" "Power symbol creates a global label with name \"GND\" , ground"
+			(at 298.45 223.52 0)
+			(effects
+				(font
+					(size 1.27 1.27)
+				)
+				(hide yes)
+			)
+		)
+		(pin "1"
+		)
+		(instances
+			(project "MouseWB5"
+				(path "/3003f723-e5bb-4cdb-ac11-d8017cbd2609"
+					(reference "#PWR0107")
+					(unit 1)
+				)
+			)
+		)
+	)
+	(symbol
+		(lib_id "power:GND")
 		(at 552.45 336.55 0)
 		(unit 1)
@@
 					(unit 1)
 				)
+			)
+		)
+	)
+	(symbol
+		(lib_id "power:+1V8")
+		(at 293.37 223.52 180)
+		(unit 1)
+		(exclude_from_sim no)
+		(in_bom yes)
+		(on_board yes)
+		(dnp no)
+		(fields_autoplaced yes)
+		(property "Reference" "#PWR0108"
+			(at 293.37 219.71 0)
+			(effects
+				(font
+					(size 1.27 1.27)
+				)
+				(hide yes)
+			)
+		)
+		(property "Value" "+1V8"
+			(at 293.37 228.6 0)
+			(effects
+				(font
+					(size 1.27 1.27)
+				)
+			)
+		)
+		(property "Footprint" ""
+			(at 293.37 223.52 0)
+			(effects
+				(font
+					(size 1.27 1.27)
+				)
+				(hide yes)
+			)
+		)
+		(property "Datasheet" ""
+			(at 293.37 223.52 0)
+			(effects
+				(font
+					(size 1.27 1.27)
+				)
+				(hide yes)
+			)
+		)
+		(property "Description" "Power symbol creates a global label with name \"+1V8\""
+			(at 293.37 223.52 0)
+			(effects
+				(font
+					(size 1.27 1.27)
+				)
+				(hide yes)
+			)
+		)
+		(pin "1"
+		)
+		(instances
+			(project "MouseWB5"
+				(path "/3003f723-e5bb-4cdb-ac11-d8017cbd2609"
+					(reference "#PWR0108")
+					(unit 1)
+				)

Commit message: work
Connections:
- net +1V8: now also U1.15 (VBAT), U1.17 (VDDSMPS), U1.32 (VDDUSB), U1.4 (VREF), U1.6 (VDDA), U2.11 (REF), U3.11 (REF), U5.5 (VDDIO), U5.8 (VDD)
- net +3V3: no longer U1.15 (VBAT), U1.17 (VDDSMPS), U1.32 (VDDUSB), U1.4 (VREF), U1.6 (VDDA), U2.11 (REF), U3.11 (REF), U5.5 (VDDIO), U5.8 (VDD)
