File: MouseWB5/MouseWB5.kicad_sch (KiCad schematic)
At the start: 71 parts, among them J1 USB_C_Receptacle_USB2.0_14P, J9 Conn_01x02_Socket, M1 Conn_01x02_Socket, M2 Conn_01x02_Socket, M3 Conn_01x02_Socket, M4 Conn_01x02_Socket, M5 Conn_01x02_Socket, Q2 CSD13380F3, SW1 SW_Push, U1 STM32WB5MMG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

Commit message: work
Parts:
- added R14, R15, R16, R17: 330mO, Resistor_SMD:R_1206_3216Metric_Pad1.30x1.75mm_HandSolder, symbol Device:R
Connections:
- net GND: now also R14.2, R15.2, R16.2, R17.2
- net SENSE_LF: now also R16.1
- net SENSE_LR: now also R17.1
- net SENSE_RF: now also R14.1
- net SENSE_RR: now also R15.1

Commit message: work
Parts:
- removed D3: BAT54J, Diode_SMD:D_SOD-323F, symbol Diode:BAT54J
- added D4: 1N5819WS, Diode_SMD:D_SOD-323, symbol Diode:1N5819WS
- added R18: 22r, Resistor_SMD:R_0201_0603Metric, symbol Device:R
- Q2: value CSD13380F3 -> MCC SI8810; footprint Package_DFN_QFN:Texas_PicoStar_DFN-3_0.69x0.60mm -> Package_TO_SOT_SMD:SOT-23
Connections:
- net +BATT: now also D4.1 (K)
- net FAN_CTRL: now also R18.2; no longer Q2.1 (G), R9.2
- net at M5.2 (Pin_2), Q2.3 (D): now also D4.2 (A)
- new net: Q2.1 (G), R18.1, R9.2
Other:
- moved on the sheet: R9
Changed lines of the file:
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@@
 	(text_box "FAN DRIVER"
 		(exclude_from_sim no)
-		(at 238.76 215.9 0)
-		(size 40.64 50.8)
+		(at 231.14 215.9 0)
+		(size 48.26 50.8)
 		(margins 0.9525 0.9525 0.9525 0.9525)
 		(stroke
@@
 	)
 	(junction
-		(at 252.73 247.65)
+		(at 251.46 247.65)
 		(diameter 0)
 		(color 0 0 0 0)
@@
 	(wire
 		(pts
+			(xy 250.19 247.65) (xy 251.46 247.65)
+		)
+		(stroke
+			(width 0)
+			(type default)
+		)
+	)
+	(wire
+		(pts
 			(xy 414.02 64.77) (xy 414.02 66.04)
 		)
@@
 	(wire
 		(pts
+			(xy 251.46 247.65) (xy 252.73 247.65)
+		)
+		(stroke
+			(width 0)
+			(type default)
+		)
+	)
+	(wire
+		(pts
 			(xy 336.55 72.39) (xy 336.55 69.85)
 		)
@@
 	(wire
 		(pts
-			(xy 242.57 247.65) (xy 252.73 247.65)
-		)
-		(stroke
-			(width 0)
-			(type default)
-		)
-	)
-	(wire
-		(pts
 			(xy 266.7 226.06) (xy 266.7 231.14)
 		)
@@
 	(wire
 		(pts
-			(xy 252.73 255.27) (xy 260.35 255.27)
+			(xy 251.46 255.27) (xy 260.35 255.27)
 		)
 		(stroke
@@
 	(wire
 		(pts
+			(xy 233.68 247.65) (xy 242.57 247.65)
+		)
+		(stroke
+			(width 0)
+			(type default)
+		)
+	)
+	(wire
+		(pts
 			(xy 356.87 242.57) (xy 347.98 242.57)
 		)
@@
 	)
 	(label "FAN_CTRL"
-		(at 242.57 247.65 0)
+		(at 233.68 247.65 0)
 		(effects
 			(font
@@
 	)
 	(symbol
-		(lib_id "Diode:BAT54J")
-		(at 252.73 232.41 270)
-		(unit 1)
-		(exclude_from_sim no)
-		(in_bom yes)
-		(on_board yes)
-		(dnp no)
-		(fields_autoplaced yes)
-		(property "Reference" "D3"
-			(at 255.27 230.8224 90)
-			(effects
-				(font
-					(size 1.27 1.27)
-				)
-				(justify left)
-			)
-		)
-		(property "Value" "BAT54J"
-			(at 255.27 233.3624 90)
-			(effects
-				(font
-					(size 1.27 1.27)
-				)
-				(justify left)
-			)
-		)
-		(property "Footprint" "Diode_SMD:D_SOD-323F"
-			(at 248.285 232.41 0)
-			(effects
-				(font
-					(size 1.27 1.27)
-				)
-				(hide yes)
-			)
-		)
-		(property "Datasheet" "https://assets.nexperia.com/documents/data-sheet/BAT54J.pdf"
-			(at 252.73 232.41 0)
-			(effects
-				(font
-					(size 1.27 1.27)
-				)
-				(hide yes)
-			)
-		)
-		(property "Description" "30V 200mA Schottky diode, SOD-323F"
-			(at 252.73 232.41 0)
-			(effects
-				(font
-					(size 1.27 1.27)
-				)
-				(hide yes)
-			)
-		)
-		(pin "1"
-		)
-		(pin "2"
-		)
-		(instances
-			(project ""
-				(path "/3003f723-e5bb-4cdb-ac11-d8017cbd2609"
-					(reference "D3")
-					(unit 1)
-				)
-			)
-		)
-	)
-	(symbol
 		(lib_id "2024-11-26_16-37-43:STBC08PMR")
 		(at 236.22 55.88 0)
@@
 	(symbol
 		(lib_id "Device:R")
-		(at 252.73 251.46 180)
+		(at 251.46 251.46 180)
 		(unit 1)
 		(exclude_from_sim no)
@@
 		(dnp no)
 		(property "Reference" "R9"
-			(at 252.73 251.206 90)
+			(at 251.46 251.206 90)
 			(effects
 				(font
@@
 		)
 		(property "Value" "20k"
-			(at 250.444 251.206 90)
+			(at 249.174 251.206 90)
 			(effects
 				(font
@@
 		)
 		(property "Footprint" "Resistor_SMD:R_0402_1005Metric"
-			(at 254.508 251.46 90)
+			(at 253.238 251.46 90)
 			(effects
 				(font
@@
 		)
 		(property "Datasheet" "~"
-			(at 252.73 251.46 0)
+			(at 251.46 251.46 0)
 			(effects
 				(font
@@
 		)
 		(property "Description" ""
-			(at 252.73 251.46 0)
+			(at 251.46 251.46 0)
 			(effects
 				(font
@@
 		)
 		(property "LCSC" "C105872"
-			(at 252.73 251.46 0)
+			(at 251.46 251.46 0)
 			(effects
 				(font
@@
 			)
 		)
-		(property "Value" "CSD13380F3"
+		(property "Value" "MCC SI8810"
 			(at 264.16 248.9199 0)
 			(effects
@@
 			)
 		)
-		(property "Footprint" "Package_DFN_QFN:Texas_PicoStar_DFN-3_0.69x0.60mm"
+		(property "Footprint" "Package_TO_SOT_SMD:SOT-23"
 			(at 262.89 249.555 0)
 			(effects
@@
 	)
 	(symbol
+		(lib_id "Diode:1N5819WS")
+		(at 252.73 232.41 270)
+		(unit 1)
+		(exclude_from_sim no)
+		(in_bom yes)
+		(on_board yes)
+		(dnp no)
+		(fields_autoplaced yes)
+		(property "Reference" "D4"
+			(at 255.27 230.8224 90)
+			(effects
+				(font
+					(size 1.27 1.27)
+				)
+				(justify left)
+			)
+		)
+		(property "Value" "1N5819WS"
+			(at 255.27 233.3624 90)
+			(effects
+				(font
+					(size 1.27 1.27)
+				)
+				(justify left)
+			)
+		)
+		(property "Footprint" "Diode_SMD:D_SOD-323"
+			(at 248.285 232.41 0)
+			(effects
+				(font
+					(size 1.27 1.27)
+				)
+				(hide yes)
+			)
+		)
+		(property "Datasheet" "https://datasheet.lcsc.com/lcsc/2204281430_Guangdong-Hottech-1N5819WS_C191023.pdf"
+			(at 252.73 232.41 0)
+			(effects
+				(font
+					(size 1.27 1.27)
+				)
+				(hide yes)
+			)
+		)
+		(property "Description" "40V 600mV@1A 1A SOD-323 Schottky Barrier Diodes, SOD-323"
+			(at 252.73 232.41 0)
+			(effects
+				(font
+					(size 1.27 1.27)
+				)
+				(hide yes)
+			)
+		)
+		(pin "1"
+		)
+		(pin "2"
+		)
+		(instances
+			(project ""
+				(path "/3003f723-e5bb-4cdb-ac11-d8017cbd2609"
+					(reference "D4")
+					(unit 1)
+				)
+			)
+		)
+	)
+	(symbol
 		(lib_id "Connector:Conn_01x02_Socket")
 		(at 328.93 128.27 270)
@@
 					(unit 1)
 				)
+			)
+		)
+	)
+	(symbol
+		(lib_id "Device:R")
+		(at 246.38 247.65 270)
+		(unit 1)
+		(exclude_from_sim no)
+		(in_bom yes)
+		(on_board yes)
+		(dnp no)
+		(property "Reference" "R18"
+			(at 245.618 247.904 90)
+			(effects
+				(font
+					(size 1.27 1.27)
+				)
+			)
+		)
+		(property "Value" "22r"
+			(at 246.38 244.856 0)
+			(effects
+				(font
+					(size 1.27 1.27)
+				)
+			)
+		)
+		(property "Footprint" "Resistor_SMD:R_0201_0603Metric"
+			(at 246.38 245.872 90)
+			(effects
+				(font
+					(size 1.27 1.27)
+				)
+				(hide yes)
+			)
+		)
+		(property "Datasheet" "~"
+			(at 246.38 247.65 0)
+			(effects
+				(font
+					(size 1.27 1.27)
+				)
+				(hide yes)
+			)
+		)
+		(property "Description" ""
+			(at 246.38 247.65 0)
+			(effects
+				(font
+					(size 1.27 1.27)
+				)
+				(hide yes)
+			)
+		)
+		(property "LCSC" "C105872"
+			(at 246.38 247.65 0)
+			(effects
+				(font
+					(size 1.27 1.27)
+				)
+				(hide yes)
+			)
+		)
+		(pin "1"
+		)
+		(pin "2"
+		)
+		(instances
+			(project "MouseWB5"
+				(path "/3003f723-e5bb-4cdb-ac11-d8017cbd2609"
+					(reference "R18")
+					(unit 1)
+				)

Commit message: work
Parts:
- D4: LCSC (none) -> C191023
- Q2: LCSC (none) -> C669009
Other:
- note added: "boot pull down R hiding here"
- moved on the sheet: D1, D2
Changed lines of the file:
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@@
 	(generator_version "9.0")
 	(paper "A2")
+	(text "boot pull down\nR hiding here"
+		(exclude_from_sim no)
+		(at 515.62 345.694 0)
+		(effects
+			(font
+				(size 1.27 1.27)
+			)
+		)
+	)
 	(text "Designed By Isaac Olson "
 		(exclude_from_sim no)
@@
 	(wire
 		(pts
-			(xy 180.34 363.22) (xy 180.34 365.76)
+			(xy 180.34 363.22) (xy 180.34 364.49)
 		)
 		(stroke
@@
 	(wire
 		(pts
+			(xy 180.34 372.11) (xy 180.34 373.38)
+		)
+		(stroke
+			(width 0)
+			(type default)
+		)
+	)
+	(wire
+		(pts
 			(xy 444.5 240.03) (xy 447.04 240.03)
 		)
@@
 	(wire
 		(pts
-			(xy 190.5 360.68) (xy 190.5 365.76)
+			(xy 190.5 360.68) (xy 190.5 364.49)
 		)
 		(stroke
@@
 	(wire
 		(pts
+			(xy 190.5 372.11) (xy 190.5 373.38)
+		)
+		(stroke
+			(width 0)
+			(type default)
+		)
+	)
+	(wire
+		(pts
 			(xy 462.28 217.17) (xy 462.28 212.09)
 		)
@@
 	(symbol
 		(lib_id "Device:LED")
-		(at 180.34 369.57 90)
+		(at 180.34 368.3 90)
 		(unit 1)
 		(exclude_from_sim no)
@@
 		(fields_autoplaced yes)
 		(property "Reference" "D1"
-			(at 184.15 369.8874 90)
+			(at 184.15 368.6174 90)
 			(effects
 				(font
@@
 		)
 		(property "Value" "LED"
-			(at 184.15 372.4274 90)
+			(at 184.15 371.1574 90)
 			(effects
 				(font
@@
 		)
 		(property "Footprint" "LED_SMD:LED_0402_1005Metric"
-			(at 180.34 369.57 0)
+			(at 180.34 368.3 0)
 			(effects
 				(font
@@
 		)
 		(property "Datasheet" "~"
-			(at 180.34 369.57 0)
+			(at 180.34 368.3 0)
 			(effects
 				(font
@@
 		)
 		(property "Description" "Light emitting diode"
-			(at 180.34 369.57 0)
+			(at 180.34 368.3 0)
 			(effects
 				(font
@@
 			)
 		)
-		(property "Datasheet" "https://www.ti.com/lit/ds/symlink/csd13380f3.pdf"
+		(property "Datasheet" ""
 			(at 262.89 251.46 0)
 			(effects
@@
 			)
 		)
-		(property "Description" "3.6A Id, 12V Vds, N-Channel MOSFET, 76mOhm Ron,max @ 4.5Vgs, 0.91nC Qg,typ @ 4.5Vgs, PicoStar 0.73x0.64mm max, 0.69x0.60mm nom"
+		(property "Description" ""
 			(at 306.07 247.65 0)
 			(effects
@@
 			)
 		)
+		(property "LCSC" "C669009"
+			(at 257.81 247.65 0)
+			(effects
+				(font
+					(size 1.27 1.27)
+				)
+				(hide yes)
+			)
+		)
 		(pin "1"
 		)
@@
 			)
 		)
+		(property "LCSC" "C191023"
+			(at 252.73 232.41 90)
+			(effects
+				(font
+					(size 1.27 1.27)
+				)
+				(hide yes)
+			)
+		)
 		(pin "1"
 		)
@@
 	(symbol
 		(lib_id "Device:LED")
-		(at 190.5 369.57 90)
+		(at 190.5 368.3 90)
 		(unit 1)
 		(exclude_from_sim no)
@@
 		(fields_autoplaced yes)
 		(property "Reference" "D2"
-			(at 194.31 369.8874 90)
+			(at 194.31 368.6174 90)
 			(effects
 				(font
@@
 		)
 		(property "Value" "LED"
-			(at 194.31 372.4274 90)
+			(at 194.31 371.1574 90)
 			(effects
 				(font
@@
 		)
 		(property "Footprint" "LED_SMD:LED_0402_1005Metric"
-			(at 190.5 369.57 0)
+			(at 190.5 368.3 0)
 			(effects
 				(font
@@
 		)
 		(property "Datasheet" "~"
-			(at 190.5 369.57 0)
+			(at 190.5 368.3 0)
 			(effects
 				(font
@@
 		)
 		(property "Description" "Light emitting diode"
-			(at 190.5 369.57 0)
+			(at 190.5 368.3 0)
 			(effects
 				(font

Commit message: work
Parts:
- C3, C6: LCSC (none) -> C602037
- LED1, LED2, LED3, LED4, LED5, LED6, LED7, LED8: LCSC (none) -> C5349953
- R14, R15, R16, R17: value 330mO -> 330mR
- SW1: LCSC (none) -> C50176685
- U4: LCSC (none) -> C2876234
- U6: LCSC (none) -> C262929
- U7: LCSC (none) -> C524780
Changed lines of the file:
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@@
 			)
 		)
+		(property "LCSC" "C262929"
+			(at 236.22 55.88 0)
+			(effects
+				(font
+					(size 1.27 1.27)
+				)
+				(hide yes)
+			)
+		)
 		(pin "2"
 		)
@@
 			)
 		)
+		(property "LCSC" "C50176685"
+			(at 311.15 186.69 0)
+			(effects
+				(font
+					(size 1.27 1.27)
+				)
+				(hide yes)
+			)
+		)
 		(pin "2"
 		)
@@
 			)
 		)
-		(property "Value" "330mO"
+		(property "Value" "330mR"
 			(at 406.4 250.1899 0)
 			(effects
@@
 			)
 		)
-		(property "Value" "330mO"
+		(property "Value" "330mR"
 			(at 406.4 262.8899 0)
 			(effects
@@
 			)
 		)
+		(property "LCSC" "C2876234"
+			(at 396.24 100.33 0)
+			(effects
+				(font
+					(size 1.27 1.27)
+				)
+				(hide yes)
+			)
+		)
 		(pin "3"
 		)
@@
 			)
 		)
+		(property "LCSC" "C5349953"
+			(at 414.02 367.03 0)
+			(effects
+				(font
+					(size 1.27 1.27)
+				)
+				(hide yes)
+			)
+		)
 		(pin "1"
 		)
@@
 			)
 		)
+		(property "LCSC" "C5349953"
+			(at 292.1 367.03 0)
+			(effects
+				(font
+					(size 1.27 1.27)
+				)
+				(hide yes)
+			)
+		)
 		(pin "1"
 		)
@@
 			)
 		)
+		(property "LCSC" "C5349953"
+			(at 265.43 367.03 0)
+			(effects
+				(font
+					(size 1.27 1.27)
+				)
+				(hide yes)
+			)
+		)
 		(pin "1"
 		)
@@
 			)
 		)
-		(property "Value" "330mO"
+		(property "Value" "330mR"
 			(at 408.94 207.0099 0)
 			(effects
@@
 			)
 		)
+		(property "LCSC" "C5349953"
+			(at 441.96 367.03 0)
+			(effects
+				(font
+					(size 1.27 1.27)
+				)
+				(hide yes)
+			)
+		)
 		(pin "1"
 		)
@@
 			)
 		)
-		(property "Value" "330mO"
+		(property "Value" "330mR"
 			(at 408.94 194.3099 0)
 			(effects
@@
 			)
 		)
+		(property "LCSC" "C602037"
+			(at 448.31 175.26 0)
+			(effects
+				(font
+					(size 1.27 1.27)
+				)
+				(hide yes)
+			)
+		)
 		(pin "1"
 		)
@@
 			)
 		)
+		(property "LCSC" "C602037"
+			(at 448.31 232.41 0)
+			(effects
+				(font
+					(size 1.27 1.27)
+				)
+				(hide yes)
+			)
+		)
 		(pin "1"
 		)
@@
 			)
 		)
+		(property "LCSC" "C5349953"
+			(at 387.35 367.03 0)
+			(effects
+				(font
+					(size 1.27 1.27)
+				)
+				(hide yes)
+			)
+		)
 		(pin "1"
 		)
@@
 			)
 		)
+		(property "LCSC" "C5349953"
+			(at 320.04 367.03 0)
+			(effects
+				(font
+					(size 1.27 1.27)
+				)
+				(hide yes)
+			)
+		)
 		(pin "1"
 		)
@@
 			)
 		)
+		(property "LCSC" "C5349953"
+			(at 361.95 367.03 0)
+			(effects
+				(font
+					(size 1.27 1.27)
+				)
+				(hide yes)
+			)
+		)
 		(pin "1"
 		)
@@
 			)
 		)
+		(property "LCSC" "C5349953"
+			(at 240.03 367.03 0)
+			(effects
+				(font
+					(size 1.27 1.27)
+				)
+				(hide yes)
+			)
+		)
 		(pin "1"
 		)
@@
 			(at 396.24 67.31 0)
 			(effects
+				(font
+					(size 1.27 1.27)
+				)
+				(hide yes)
+			)
+		)
+		(property "LCSC" "C524780"
+			(at 396.24 67.31 0)
+			(effects

Commit message: work
Parts:
- added C11, C12: 22nF, Capacitor_SMD:C_0402_1005Metric, symbol Device:C
Connections:
- net +BATT: now also C11.1, C12.1
- net GND: now also C11.2, C12.2

Commit message: work
Parts:
- added C13, C14: 1nF, Capacitor_SMD:C_0402_1005Metric, symbol Device:C
- added C15, C16: 10nF, Capacitor_SMD:C_0402_1005Metric, symbol Device:C
- added R19, R20: 20k, Resistor_SMD:R_0402_1005Metric, symbol Device:R
Connections:
- net +1V8: now also R19.2, R20.2
- net GND: now also C13.1, C14.1, C15.1, C16.1
- net L_EN: now also C13.2
- net L_RESET: now also C16.2, R19.1
- net R_EN: now also C14.2
- net R_RESET: now also C15.2, R20.1

Commit message: work
Parts:
- added C17, C18: 40nF, Capacitor_SMD:C_0402_1005Metric, symbol Device:C
- added R21, R24: 33k, Resistor_SMD:R_0402_1005Metric, symbol Device:R
- added R22, R23: 11k, Resistor_SMD:R_0402_1005Metric, symbol Device:R
- C13, C14: value 1nF -> 10nF
- C15, C16: value 10nF -> 1nF
- R19: LCSC C105872 -> (none)
Connections:
- net GND: now also C17.2, C18.2, R22.1, R23.1
- net L_REF: now also R21.2; no longer U2.11 (REF)
- net R_REF: now also R24.2; no longer U3.11 (REF)
- new net: C17.1, R21.1, R22.2, U2.11 (REF)
- new net: C18.1, R23.2, R24.1, U3.11 (REF)

Commit message: work
Other:
- note added: "boot pull down R hiding here on board"
- note removed: "boot pull down R hiding here"
Changed lines of the file:
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@@
 	(generator_version "9.0")
 	(paper "A2")
-	(text "boot pull down\nR hiding here"
+	(text "boot pull down\nR hiding here\non board"
 		(exclude_from_sim no)
 		(at 515.62 345.694 0)
