File: MouseWB5/MouseWB5.kicad_sch (KiCad schematic)
At the start: 90 parts, among them J1 USB_C_Receptacle_USB2.0_14P, J9 Conn_01x02_Socket, M1 Conn_01x02_Socket, M2 Conn_01x02_Socket, M3 Conn_01x02_Socket, M4 Conn_01x02_Socket, M5 Conn_01x02_Socket, Q2 MCC SI8810, SW1 SW_Push, U1 STM32WB5MMG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

Commit message: exp3_done
Parts:
- C19, C2, C20: LCSC C2168305 -> C1525
Changed lines of the file:
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@@
 			)
 		)
-		(property "LCSC" "C2168305"
+		(property "LCSC" "C1525"
 			(at 400.05 359.41 0)
 			(effects
@@
 			)
 		)
-		(property "LCSC" "C2168305"
+		(property "LCSC" "C1525"
 			(at 373.38 360.68 0)
 			(effects
@@
 			)
 		)
-		(property "LCSC" "C2168305"
+		(property "LCSC" "C1525"
 			(at 419.1 298.45 0)
 			(effects

Commit message: work
Parts:
- R21, R24: value 33k -> 22k; LCSC C138003 -> C82868
Changed lines of the file:
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@@
 			)
 		)
-		(property "Value" "33k"
+		(property "Value" "22k"
 			(at 496.824 268.224 90)
 			(effects
@@
 			)
 		)
-		(property "LCSC" "C138003"
+		(property "LCSC" "C82868"
 			(at 496.57 270.51 0)
 			(effects
@@
 			)
 		)
-		(property "Value" "33k"
+		(property "Value" "22k"
 			(at 498.094 212.344 90)
 			(effects
@@
 			)
 		)
-		(property "LCSC" "C138003"
+		(property "LCSC" "C82868"
 			(at 497.84 214.63 0)
 			(effects

Commit message: work
Connections:
- net GND: now also I2C1_HEADER1.8 (Pin_8), I2C3_HEADER1.8 (Pin_8), SPI2_HEADER1.10 (Pin_10)
Changed lines of the file:
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@@
 	(symbol
 		(lib_id "power:GND")
+		(at 205.74 298.45 270)
+		(unit 1)
+		(exclude_from_sim no)
+		(in_bom yes)
+		(on_board yes)
+		(dnp no)
+		(fields_autoplaced yes)
+		(property "Reference" "#PWR0134"
+			(at 199.39 298.45 0)
+			(effects
+				(font
+					(size 1.27 1.27)
+				)
+				(hide yes)
+			)
+		)
+		(property "Value" "GND"
+			(at 201.93 298.4499 90)
+			(effects
+				(font
+					(size 1.27 1.27)
+				)
+				(justify right)
+			)
+		)
+		(property "Footprint" ""
+			(at 205.74 298.45 0)
+			(effects
+				(font
+					(size 1.27 1.27)
+				)
+				(hide yes)
+			)
+		)
+		(property "Datasheet" ""
+			(at 205.74 298.45 0)
+			(effects
+				(font
+					(size 1.27 1.27)
+				)
+				(hide yes)
+			)
+		)
+		(property "Description" "Power symbol creates a global label with name \"GND\" , ground"
+			(at 205.74 298.45 0)
+			(effects
+				(font
+					(size 1.27 1.27)
+				)
+				(hide yes)
+			)
+		)
+		(pin "1"
+		)
+		(instances
+			(project "MouseWB5"
+				(path "/3003f723-e5bb-4cdb-ac11-d8017cbd2609"
+					(reference "#PWR0134")
+					(unit 1)
+				)
+			)
+		)
+	)
+	(symbol
+		(lib_id "power:GND")
 		(at 163.83 280.67 270)
 		(unit 1)
@@
 	)
 	(symbol
+		(lib_id "power:GND")
+		(at 247.65 298.45 270)
+		(unit 1)
+		(exclude_from_sim no)
+		(in_bom yes)
+		(on_board yes)
+		(dnp no)
+		(fields_autoplaced yes)
+		(property "Reference" "#PWR0133"
+			(at 241.3 298.45 0)
+			(effects
+				(font
+					(size 1.27 1.27)
+				)
+				(hide yes)
+			)
+		)
+		(property "Value" "GND"
+			(at 243.84 298.4499 90)
+			(effects
+				(font
+					(size 1.27 1.27)
+				)
+				(justify right)
+			)
+		)
+		(property "Footprint" ""
+			(at 247.65 298.45 0)
+			(effects
+				(font
+					(size 1.27 1.27)
+				)
+				(hide yes)
+			)
+		)
+		(property "Datasheet" ""
+			(at 247.65 298.45 0)
+			(effects
+				(font
+					(size 1.27 1.27)
+				)
+				(hide yes)
+			)
+		)
+		(property "Description" "Power symbol creates a global label with name \"GND\" , ground"
+			(at 247.65 298.45 0)
+			(effects
+				(font
+					(size 1.27 1.27)
+				)
+				(hide yes)
+			)
+		)
+		(pin "1"
+		)
+		(instances
+			(project "MouseWB5"
+				(path "/3003f723-e5bb-4cdb-ac11-d8017cbd2609"
+					(reference "#PWR0133")
+					(unit 1)
+				)
+			)
+		)
+	)
+	(symbol
 		(lib_id "power:+BATT")
 		(at 163.83 306.07 90)
@@
 					(unit 1)
 				)
+			)
+		)
+	)
+	(symbol
+		(lib_id "power:GND")
+		(at 163.83 303.53 270)
+		(unit 1)
+		(exclude_from_sim no)
+		(in_bom yes)
+		(on_board yes)
+		(dnp no)
+		(fields_autoplaced yes)
+		(property "Reference" "#PWR0135"
+			(at 157.48 303.53 0)
+			(effects
+				(font
+					(size 1.27 1.27)
+				)
+				(hide yes)
+			)
+		)
+		(property "Value" "GND"
+			(at 160.02 303.5299 90)
+			(effects
+				(font
+					(size 1.27 1.27)
+				)
+				(justify right)
+			)
+		)
+		(property "Footprint" ""
+			(at 163.83 303.53 0)
+			(effects
+				(font
+					(size 1.27 1.27)
+				)
+				(hide yes)
+			)
+		)
+		(property "Datasheet" ""
+			(at 163.83 303.53 0)
+			(effects
+				(font
+					(size 1.27 1.27)
+				)
+				(hide yes)
+			)
+		)
+		(property "Description" "Power symbol creates a global label with name \"GND\" , ground"
+			(at 163.83 303.53 0)
+			(effects
+				(font
+					(size 1.27 1.27)
+				)
+				(hide yes)
+			)
+		)
+		(pin "1"
+		)
+		(instances
+			(project "MouseWB5"
+				(path "/3003f723-e5bb-4cdb-ac11-d8017cbd2609"
+					(reference "#PWR0135")
+					(unit 1)
+				)

Commit message: work
Connections:
- net I2C2_GPIO renamed I2C3_GPIO
Changed lines of the file:
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@@
 		)
 	)
-	(label "I2C2_GPIO"
+	(label "I2C3_GPIO"
 		(at 237.49 295.91 0)
 		(effects
@@
 		)
 	)
-	(label "I2C2_GPIO"
+	(label "I2C3_GPIO"
 		(at 359.41 265.43 180)
 		(effects

Commit message: work
Parts:
- added C21, C22: 10u, Capacitor_SMD:C_0805_2012Metric, symbol Device:C
- added MR3: 5.1k, Resistor_SMD:R_0402_1005Metric, symbol Device:R
- added R3, R4: 20k, Resistor_SMD:R_0402_1005Metric, symbol Device:R
- C11, C12: value 22nF -> 2.2uf; LCSC C337699 -> C170151
Connections:
- net +1V8: now also R3.2, R4.2
- net +BATT: now also C21.1, C22.1
- net GND: now also C21.2, C22.2, MR3.1, MR3.2
- net L_EN: now also R3.1
- net R_EN: now also R4.1
Other:
- note removed: "boot pull down R hiding here on board"

Commit message: work
Connections:
- net GND: now also U1.58 (ANT_IN), U1.59 (RF_OUT)
- no-connect marks 29 -> 27
Changed lines of the file:
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@@
 	)
 	(junction
+		(at 347.98 275.59)
+		(diameter 0)
+		(color 0 0 0 0)
+	)
+	(junction
 		(at 414.02 97.79)
 		(diameter 0)
@@
 	)
 	(no_connect
-		(at 347.98 273.05)
-	)
-	(no_connect
-		(at 347.98 275.59)
-	)
-	(no_connect
 		(at 247.65 298.45)
 	)
@@
 	(wire
 		(pts
+			(xy 347.98 275.59) (xy 347.98 276.86)
+		)
+		(stroke
+			(width 0)
+			(type default)
+		)
+	)
+	(wire
+		(pts
 			(xy 444.5 201.93) (xy 453.39 201.93)
 		)
@@
 	(wire
 		(pts
+			(xy 347.98 273.05) (xy 347.98 275.59)
+		)
+		(stroke
+			(width 0)
+			(type default)
+		)
+	)
+	(wire
+		(pts
 			(xy 353.06 240.03) (xy 347.98 240.03)
 		)
@@
 					(unit 1)
 				)
+			)
+		)
+	)
+	(symbol
+		(lib_id "power:GND")
+		(at 347.98 276.86 0)
+		(unit 1)
+		(exclude_from_sim no)
+		(in_bom yes)
+		(on_board yes)
+		(dnp no)
+		(property "Reference" "#PWR0142"
+			(at 347.98 283.21 0)
+			(effects
+				(font
+					(size 1.27 1.27)
+				)
+				(hide yes)
+			)
+		)
+		(property "Value" "GND"
+			(at 347.98 280.67 0)
+			(effects
+				(font
+					(size 1.27 1.27)
+				)
+			)
+		)
+		(property "Footprint" ""
+			(at 347.98 276.86 0)
+			(effects
+				(font
+					(size 1.27 1.27)
+				)
+				(hide yes)
+			)
+		)
+		(property "Datasheet" ""
+			(at 347.98 276.86 0)
+			(effects
+				(font
+					(size 1.27 1.27)
+				)
+				(hide yes)
+			)
+		)
+		(property "Description" "Power symbol creates a global label with name \"GND\" , ground"
+			(at 347.98 276.86 0)
+			(effects
+				(font
+					(size 1.27 1.27)
+				)
+				(hide yes)
+			)
+		)
+		(pin "1"
+		)
+		(instances
+			(project "MouseWB5"
+				(path "/3003f723-e5bb-4cdb-ac11-d8017cbd2609"
+					(reference "#PWR0142")
+					(unit 1)
+				)

Commit message: work
Parts:
- R10: LCSC C93942 -> C4109
- R14, R15, R16, R17: LCSC C7467250 -> C2932844
Changed lines of the file:
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@@
 			)
 		)
-		(property "LCSC" "C7467250"
+		(property "LCSC" "C2932844"
 			(at 403.86 248.92 0)
 			(effects
@@
 			)
 		)
-		(property "LCSC" "C7467250"
+		(property "LCSC" "C2932844"
 			(at 403.86 261.62 0)
 			(effects
@@
 			)
 		)
-		(property "LCSC" "C93942"
+		(property "LCSC" "C4109"
 			(at 285.75 60.96 90)
 			(effects
@@
 			)
 		)
-		(property "LCSC" "C7467250"
+		(property "LCSC" "C2932844"
 			(at 406.4 205.74 0)
 			(effects
@@
 			)
 		)
-		(property "LCSC" "C7467250"
+		(property "LCSC" "C2932844"
 			(at 406.4 193.04 0)
 			(effects

Commit message: work
Parts:
- M1, M2, M3, M4, M5: footprint Connector_JST:JST_SH_BM02B-SRSS-TB_1x02-1MP_P1.00mm_Vertical -> Connector_JST:JST_GH_BM02B-GHS-TBT_1x02-1MP_P1.25mm_Vertical; LCSC C160388 -> C161690
- U5: LCSC C2655100 -> C481766
Changed lines of the file:
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@@
 			)
 		)
-		(property "LCSC" "C2655100"
+		(property "LCSC" "C481766"
 			(at 434.34 316.23 0)
 			(effects
@@
 			)
 		)
-		(property "Footprint" "Connector_JST:JST_SH_BM02B-SRSS-TB_1x02-1MP_P1.00mm_Vertical"
+		(property "Footprint" "Connector_JST:JST_GH_BM02B-GHS-TBT_1x02-1MP_P1.25mm_Vertical"
 			(at 411.48 252.73 0)
 			(effects
@@
 			)
 		)
-		(property "LCSC" "C160388"
+		(property "LCSC" "C161690"
 			(at 411.48 252.73 0)
 			(effects
@@
 			)
 		)
-		(property "Footprint" "Connector_JST:JST_SH_BM02B-SRSS-TB_1x02-1MP_P1.00mm_Vertical"
+		(property "Footprint" "Connector_JST:JST_GH_BM02B-GHS-TBT_1x02-1MP_P1.25mm_Vertical"
 			(at 411.48 186.69 0)
 			(effects
@@
 			)
 		)
-		(property "LCSC" "C160388"
+		(property "LCSC" "C161690"
 			(at 411.48 186.69 0)
 			(effects
@@
 			)
 		)
-		(property "Footprint" "Connector_JST:JST_SH_BM02B-SRSS-TB_1x02-1MP_P1.00mm_Vertical"
+		(property "Footprint" "Connector_JST:JST_GH_BM02B-GHS-TBT_1x02-1MP_P1.25mm_Vertical"
 			(at 411.48 196.85 0)
 			(effects
@@
 			)
 		)
-		(property "LCSC" "C160388"
+		(property "LCSC" "C161690"
 			(at 411.48 196.85 0)
 			(effects
@@
 			)
 		)
-		(property "Footprint" "Connector_JST:JST_SH_BM02B-SRSS-TB_1x02-1MP_P1.00mm_Vertical"
+		(property "Footprint" "Connector_JST:JST_GH_BM02B-GHS-TBT_1x02-1MP_P1.25mm_Vertical"
 			(at 271.78 231.14 0)
 			(effects
@@
 			)
 		)
-		(property "LCSC" "C160388"
+		(property "LCSC" "C161690"
 			(at 271.78 231.14 90)
 			(effects
@@
 			)
 		)
-		(property "Footprint" "Connector_JST:JST_SH_BM02B-SRSS-TB_1x02-1MP_P1.00mm_Vertical"
+		(property "Footprint" "Connector_JST:JST_GH_BM02B-GHS-TBT_1x02-1MP_P1.25mm_Vertical"
 			(at 411.48 242.57 0)
 			(effects
@@
 			)
 		)
-		(property "LCSC" "C160388"
+		(property "LCSC" "C161690"
 			(at 411.48 242.57 0)
 			(effects
