File: Board/MouseWB5.kicad_pcb (KiCad board)
At the start: 6 copper layers, 65.5 x 40 mm, 96 parts, among them J1 USB_C_Receptacle_USB2.0_14P, J9 Conn_01x02_Socket, M1 Conn_01x02_Socket, M2 Conn_01x02_Socket, M3 Conn_01x02_Socket, M4 Conn_01x02_Socket, M5 Conn_01x02_Socket, Q2 MCC SI8810, SW1 SW_Push, U1 STM32WB5MMG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

Commit message: work
Routing:
- net GND: track 170.8 -> 171.3 mm, vias 71 -> 72
Changed lines of the file:
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@@
 			(pintype "power_in")
 		)
-		(pad "7" thru_hole circle
-			(at 0 -0.55 180)
-			(size 0.5 0.5)
-			(drill 0.2)
-			(property pad_prop_heatsink)
-			(layers "*.Cu")
-			(remove_unused_layers no)
-			(net 36 "GND")
-			(pinfunction "EP")
-			(pintype "passive")
-		)
 		(pad "7" smd rect
 			(at 0 0 180)
@@
 			(zone_connect 2)
 		)
-		(pad "7" thru_hole circle
-			(at 0 0.55 180)
-			(size 0.5 0.5)
-			(drill 0.2)
-			(property pad_prop_heatsink)
-			(layers "*.Cu")
-			(remove_unused_layers no)
-			(net 36 "GND")
-			(pinfunction "EP")
-			(pintype "passive")
-		)
 		(embedded_fonts no)
 		(model "${KICAD9_3DMODEL_DIR}/Package_SON.3dshapes/WSON-6-1EP_2x2mm_P0.65mm_EP1x1.6mm.step"
@@
 			(pintype "power_in")
 		)
-		(pad "7" thru_hole circle
-			(at 0 -0.55 180)
-			(size 0.5 0.5)
-			(drill 0.2)
-			(property pad_prop_heatsink)
-			(layers "*.Cu")
-			(remove_unused_layers no)
-			(net 36 "GND")
-			(pinfunction "EP")
-			(pintype "passive")
-		)
 		(pad "7" smd rect
 			(at 0 0 180)
@@
 			(zone_connect 2)
 		)
-		(pad "7" thru_hole circle
-			(at 0 0.55 180)
-			(size 0.5 0.5)
-			(drill 0.2)
-			(property pad_prop_heatsink)
-			(layers "*.Cu")
-			(remove_unused_layers no)
-			(net 36 "GND")
-			(pinfunction "EP")
-			(pintype "passive")
-		)
 		(embedded_fonts no)
 		(model "${KICAD9_3DMODEL_DIR}/Package_SON.3dshapes/WSON-6-1EP_2x2mm_P0.65mm_EP1x1.6mm.wrl"
@@
 	)
 	(segment
-		(start 106.225 132.4)
-		(end 106.289023 132.4)
-		(width 0.2)
-		(layer "F.Cu")
-		(net 36)
-	)
-	(segment
 		(start 130.5 100.75)
 		(end 130.3 100.75)
@@
 	)
 	(segment
-		(start 106.289023 132.4)
-		(end 106.414021 132.275002)
-		(width 0.2)
-		(layer "F.Cu")
-		(net 36)
-	)
-	(segment
 		(start 101.0751 108.0751)
 		(end 101.0751 106.8251)
@@
 	)
 	(segment
+		(start 106.422039 132.275)
+		(end 106.65 132.275)
+		(width 0.2)
+		(layer "F.Cu")
+		(net 36)
+	)
+	(segment
 		(start 118.27 108.5)
 		(end 118 108.77)
@@
 	)
 	(segment
-		(start 106.418031 132.270992)
-		(end 106.414021 132.275002)
-		(width 0.2)
-		(layer "F.Cu")
-		(net 36)
-	)
-	(segment
 		(start 107 113.45)
 		(end 107.751 114.201)
@@
 	)
 	(segment
+		(start 106.65 132.275)
+		(end 106.414023 132.275)
+		(width 0.2)
+		(layer "F.Cu")
+		(net 36)
+	)
+	(segment
 		(start 128.851 109.031)
 		(end 128.3 108.48)
@@
 	)
 	(segment
+		(start 106.289023 132.4)
+		(end 106.225 132.4)
+		(width 0.2)
+		(layer "F.Cu")
+		(net 36)
+	)
+	(segment
 		(start 133.25 102.2)
 		(end 132.55 101.5)
@@
 	)
 	(segment
+		(start 106.414023 132.275)
+		(end 106.289023 132.4)
+		(width 0.2)
+		(layer "F.Cu")
+		(net 36)
+	)
+	(segment
 		(start 159.275 105.6)
 		(end 159.275 105.295)
@@
 	)
 	(segment
+		(start 106.418031 132.270992)
+		(end 106.422039 132.275)
+		(width 0.2)
+		(layer "F.Cu")
+		(net 36)
+	)
+	(segment
 		(start 120.25 119.0875)
 		(end 120.25 119.5)
@@
 	)
 	(segment
-		(start 106.418031 132.270992)
-		(end 106.414021 132.275002)
-		(width 0.2)
-		(layer "F.Cu")
-		(net 36)
-	)
-	(segment
 		(start 135.350707 133.249293)
 		(end 135.479 133.121)
@@
 	)
 	(via
-		(at 106.414021 132.275002)
-		(size 0.45)
+		(at 106.65 132.275)
+		(size 0.6)
 		(drill 0.3)
 		(layers "F.Cu" "B.Cu")
@@
 	)
 	(via
-		(at 116.5 118.5)
+		(at 115.5 117.75)
 		(size 0.6)
 		(drill 0.3)
@@
 		(drill 0.3)
 		(layers "F.Cu" "B.Cu")
+		(net 36)
+	)
+	(via
+		(at 112.6125 123.9)
+		(size 0.55)
+		(drill 0.3)
+		(layers "F.Cu" "B.Cu")

Commit message: Revert "work"
This reverts commit ebc5c044978ddb65968714e0a5620810b6ad0afb.
Routing:
- net GND: track 171.3 -> 170.8 mm, vias 72 -> 71
Changed lines of the file:
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@@
 			(pintype "power_in")
 		)
+		(pad "7" thru_hole circle
+			(at 0 -0.55 180)
+			(size 0.5 0.5)
+			(drill 0.2)
+			(property pad_prop_heatsink)
+			(layers "*.Cu")
+			(remove_unused_layers no)
+			(net 36 "GND")
+			(pinfunction "EP")
+			(pintype "passive")
+		)
 		(pad "7" smd rect
 			(at 0 0 180)
@@
 			(zone_connect 2)
 		)
+		(pad "7" thru_hole circle
+			(at 0 0.55 180)
+			(size 0.5 0.5)
+			(drill 0.2)
+			(property pad_prop_heatsink)
+			(layers "*.Cu")
+			(remove_unused_layers no)
+			(net 36 "GND")
+			(pinfunction "EP")
+			(pintype "passive")
+		)
 		(embedded_fonts no)
 		(model "${KICAD9_3DMODEL_DIR}/Package_SON.3dshapes/WSON-6-1EP_2x2mm_P0.65mm_EP1x1.6mm.step"
@@
 			(pintype "power_in")
 		)
+		(pad "7" thru_hole circle
+			(at 0 -0.55 180)
+			(size 0.5 0.5)
+			(drill 0.2)
+			(property pad_prop_heatsink)
+			(layers "*.Cu")
+			(remove_unused_layers no)
+			(net 36 "GND")
+			(pinfunction "EP")
+			(pintype "passive")
+		)
 		(pad "7" smd rect
 			(at 0 0 180)
@@
 			(zone_connect 2)
 		)
+		(pad "7" thru_hole circle
+			(at 0 0.55 180)
+			(size 0.5 0.5)
+			(drill 0.2)
+			(property pad_prop_heatsink)
+			(layers "*.Cu")
+			(remove_unused_layers no)
+			(net 36 "GND")
+			(pinfunction "EP")
+			(pintype "passive")
+		)
 		(embedded_fonts no)
 		(model "${KICAD9_3DMODEL_DIR}/Package_SON.3dshapes/WSON-6-1EP_2x2mm_P0.65mm_EP1x1.6mm.wrl"
@@
 	)
 	(segment
+		(start 106.225 132.4)
+		(end 106.289023 132.4)
+		(width 0.2)
+		(layer "F.Cu")
+		(net 36)
+	)
+	(segment
 		(start 130.5 100.75)
 		(end 130.3 100.75)
@@
 	)
 	(segment
+		(start 106.289023 132.4)
+		(end 106.414021 132.275002)
+		(width 0.2)
+		(layer "F.Cu")
+		(net 36)
+	)
+	(segment
 		(start 101.0751 108.0751)
 		(end 101.0751 106.8251)
@@
 	)
 	(segment
-		(start 106.422039 132.275)
-		(end 106.65 132.275)
-		(width 0.2)
-		(layer "F.Cu")
-		(net 36)
-	)
-	(segment
 		(start 118.27 108.5)
 		(end 118 108.77)
@@
 	)
 	(segment
+		(start 106.418031 132.270992)
+		(end 106.414021 132.275002)
+		(width 0.2)
+		(layer "F.Cu")
+		(net 36)
+	)
+	(segment
 		(start 107 113.45)
 		(end 107.751 114.201)
@@
 	)
 	(segment
-		(start 106.65 132.275)
-		(end 106.414023 132.275)
-		(width 0.2)
-		(layer "F.Cu")
-		(net 36)
-	)
-	(segment
 		(start 128.851 109.031)
 		(end 128.3 108.48)
@@
 	)
 	(segment
-		(start 106.289023 132.4)
-		(end 106.225 132.4)
-		(width 0.2)
-		(layer "F.Cu")
-		(net 36)
-	)
-	(segment
 		(start 133.25 102.2)
 		(end 132.55 101.5)
@@
 	)
 	(segment
-		(start 106.414023 132.275)
-		(end 106.289023 132.4)
-		(width 0.2)
-		(layer "F.Cu")
-		(net 36)
-	)
-	(segment
 		(start 159.275 105.6)
 		(end 159.275 105.295)
@@
 	)
 	(segment
-		(start 106.418031 132.270992)
-		(end 106.422039 132.275)
-		(width 0.2)
-		(layer "F.Cu")
-		(net 36)
-	)
-	(segment
 		(start 120.25 119.0875)
 		(end 120.25 119.5)
@@
 	)
 	(segment
+		(start 106.418031 132.270992)
+		(end 106.414021 132.275002)
+		(width 0.2)
+		(layer "F.Cu")
+		(net 36)
+	)
+	(segment
 		(start 135.350707 133.249293)
 		(end 135.479 133.121)
@@
 	)
 	(via
-		(at 106.65 132.275)
-		(size 0.6)
+		(at 106.414021 132.275002)
+		(size 0.45)
 		(drill 0.3)
 		(layers "F.Cu" "B.Cu")
@@
 	)
 	(via
-		(at 115.5 117.75)
+		(at 116.5 118.5)
 		(size 0.6)
 		(drill 0.3)
@@
 		(drill 0.3)
 		(layers "F.Cu" "B.Cu")
-		(net 36)
-	)
-	(via
-		(at 112.6125 123.9)
-		(size 0.55)
-		(drill 0.3)
-		(layers "F.Cu" "B.Cu")

Commit message: holes
Routing:
- net GND: track 170.8 -> 173.4 mm, vias 71 -> 73
Changed lines of the file:
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@@
 			(pintype "power_in")
 		)
-		(pad "7" thru_hole circle
-			(at 0 -0.55 180)
-			(size 0.5 0.5)
-			(drill 0.2)
-			(property pad_prop_heatsink)
-			(layers "*.Cu")
-			(remove_unused_layers no)
-			(net 36 "GND")
-			(pinfunction "EP")
-			(pintype "passive")
-		)
 		(pad "7" smd rect
 			(at 0 0 180)
@@
 			(zone_connect 2)
 		)
-		(pad "7" thru_hole circle
-			(at 0 0.55 180)
-			(size 0.5 0.5)
-			(drill 0.2)
-			(property pad_prop_heatsink)
-			(layers "*.Cu")
-			(remove_unused_layers no)
-			(net 36 "GND")
-			(pinfunction "EP")
-			(pintype "passive")
-		)
 		(embedded_fonts no)
 		(model "${KICAD9_3DMODEL_DIR}/Package_SON.3dshapes/WSON-6-1EP_2x2mm_P0.65mm_EP1x1.6mm.step"
@@
 			(pintype "power_in")
 		)
-		(pad "7" thru_hole circle
-			(at 0 -0.55 180)
-			(size 0.5 0.5)
-			(drill 0.2)
-			(property pad_prop_heatsink)
-			(layers "*.Cu")
-			(remove_unused_layers no)
-			(net 36 "GND")
-			(pinfunction "EP")
-			(pintype "passive")
-		)
 		(pad "7" smd rect
 			(at 0 0 180)
@@
 			(zone_connect 2)
 		)
-		(pad "7" thru_hole circle
-			(at 0 0.55 180)
-			(size 0.5 0.5)
-			(drill 0.2)
-			(property pad_prop_heatsink)
-			(layers "*.Cu")
-			(remove_unused_layers no)
-			(net 36 "GND")
-			(pinfunction "EP")
-			(pintype "passive")
-		)
 		(embedded_fonts no)
 		(model "${KICAD9_3DMODEL_DIR}/Package_SON.3dshapes/WSON-6-1EP_2x2mm_P0.65mm_EP1x1.6mm.wrl"
@@
 	)
 	(via
+		(at 115.5 116.275)
+		(size 0.6)
+		(drill 0.3)
+		(layers "F.Cu" "B.Cu")
+		(net 36)
+	)
+	(via
 		(at 125.3 103.6)
 		(size 0.6)
@@
 	)
 	(via
+		(at 112.596 123.9)
+		(size 0.6)
+		(drill 0.3)
+		(layers "F.Cu" "B.Cu")
+		(net 36)
+	)
+	(via
 		(at 116.5 118.5)
 		(size 0.6)
@@
 		(net 36)
 	)
+	(segment
+		(start 115 123.5)
+		(end 112.996 123.5)
+		(width 0.6)
+		(layer "B.Cu")
+		(net 36)
+	)
+	(segment
+		(start 112.996 123.5)
+		(end 112.596 123.9)
+		(width 0.6)
+		(layer "B.Cu")
+		(net 36)
+	)

Commit message: retouchshuntR
Parts:
- moved R16 0.25 mm to (142.8, 109.8)
- moved R17 0.25 mm to (140.2, 109.8)
Routing:
- net GND: track 173.4 -> 175.8 mm, vias 73 -> 74

Commit message: macfont
Parts:
- moved G*** 0.40 mm to (149.8, 127.0)
