File: Board/MouseWB5.kicad_pcb (KiCad board)
At the start: 6 copper layers, 65.5 x 40 mm, 96 parts, among them J1 USB_C_Receptacle_USB2.0_14P, J9 Conn_01x02_Socket, M1 Conn_01x02_Socket, M2 Conn_01x02_Socket, M3 Conn_01x02_Socket, M4 Conn_01x02_Socket, M5 Conn_01x02_Socket, Q2 MCC SI8810, SW1 SW_Push, U1 STM32WB5MMG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

Commit message: work
Routing:
- net GND: track 175.8 -> 187.3 mm

Commit message: real_order
Routing:
- net GND: track 187.3 -> 188.8 mm
Changed lines of the file:
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@@
 	(segment
 		(start 118.95555 128.245)
-		(end 118.15555 127.445)
-		(width 0.2)
-		(layer "F.Cu")
-		(net 18)
-	)
-	(segment
-		(start 118.15555 127.445)
-		(end 114.83062 127.445)
-		(width 0.2)
-		(layer "F.Cu")
-		(net 18)
-	)
-	(segment
-		(start 142.651 119.9161)
-		(end 142.651 127.4161)
+		(end 127.981407 128.245)
 		(width 0.2)
 		(layer "F.Cu")
@@
 	)
 	(segment
-		(start 114.83062 127.445)
-		(end 114.26281 128.01281)
+		(start 149.0671 113.5)
+		(end 149.5 113.5)
 		(width 0.2)
 		(layer "F.Cu")
@@
 	)
 	(segment
-		(start 140.8651 129.202)
-		(end 128.938407 129.202)
+		(start 111.67562 130.6)
+		(end 114.83062 127.445)
 		(width 0.2)
 		(layer "F.Cu")
@@
 	)
 	(segment
-		(start 111.67562 130.6)
-		(end 109.85 130.6)
+		(start 142.651 127.4161)
+		(end 142.651 119.9161)
 		(width 0.2)
 		(layer "F.Cu")
@@
 	)
 	(segment
-		(start 142.651 127.4161)
-		(end 140.8651 129.202)
+		(start 118.15555 127.445)
+		(end 118.95555 128.245)
 		(width 0.2)
 		(layer "F.Cu")
@@
 	)
 	(segment
-		(start 114.38781 127.88781)
-		(end 114.26281 128.01281)
+		(start 109.85 130.6)
+		(end 111.67562 130.6)
 		(width 0.2)
 		(layer "F.Cu")
@@
 	)
 	(segment
-		(start 128.938407 129.202)
-		(end 127.981407 128.245)
+		(start 127.981407 128.245)
+		(end 128.938407 129.202)
 		(width 0.2)
 		(layer "F.Cu")
@@
 	)
 	(segment
-		(start 114.26281 128.01281)
-		(end 111.67562 130.6)
+		(start 142.651 119.9161)
+		(end 149.0671 113.5)
 		(width 0.2)
 		(layer "F.Cu")
@@
 	)
 	(segment
-		(start 127.981407 128.245)
-		(end 118.95555 128.245)
+		(start 114.83062 127.445)
+		(end 118.15555 127.445)
 		(width 0.2)
 		(layer "F.Cu")
@@
 	)
 	(segment
-		(start 149.5 113.5)
-		(end 149.0671 113.5)
+		(start 140.8651 129.202)
+		(end 142.651 127.4161)
 		(width 0.2)
 		(layer "F.Cu")
@@
 	)
 	(segment
-		(start 149.0671 113.5)
-		(end 142.651 119.9161)
+		(start 128.938407 129.202)
+		(end 140.8651 129.202)
 		(width 0.2)
 		(layer "F.Cu")
@@
 	)
 	(segment
-		(start 106.545225 132.266322)
-		(end 106.545225 132.159624)
-		(width 0.2)
-		(layer "F.Cu")
-		(net 36)
-	)
-	(segment
 		(start 120.75 119.0875)
 		(end 120.75 120)
@@
 	)
 	(segment
-		(start 106.545225 132.266322)
-		(end 106.545225 132.159624)
-		(width 0.2)
-		(layer "F.Cu")
-		(net 36)
-	)
-	(segment
 		(start 130.02 101.03)
 		(end 130.25 100.8)
@@
 	)
 	(segment
+		(start 107.116322 132.266322)
+		(end 106.422701 132.266322)
+		(width 0.2)
+		(layer "F.Cu")
+		(net 36)
+	)
+	(segment
 		(start 141.45 111.3)
 		(end 140 111.3)
@@
 	)
 	(segment
+		(start 107.125 132.275)
+		(end 106.553903 132.275)
+		(width 0.2)
+		(layer "F.Cu")
+		(net 36)
+	)
+	(segment
 		(start 108.199 134.801)
 		(end 108.449 134.801)
@@
 	)
 	(segment
-		(start 106.545225 132.266322)
-		(end 106.422701 132.266322)
-		(width 0.2)
-		(layer "F.Cu")
-		(net 36)
-	)
-	(segment
 		(start 101.0751 103.5751)
 		(end 101 103.5)
@@
 	)
 	(segment
+		(start 107.009624 132.159624)
+		(end 106.545225 132.159624)
+		(width 0.2)
+		(layer "F.Cu")
+		(net 36)
+	)
+	(segment
 		(start 109.374 128.901)
 		(end 109.374 132.8089)
@@
 	)
 	(segment
+		(start 106.553903 132.275)
+		(end 106.483909 132.205006)
+		(width 0.2)
+		(layer "F.Cu")
+		(net 36)
+	)
+	(segment
 		(start 119.25 134.5)
 		(end 118.112911 134.5)
@@
 	)
 	(segment
-		(start 106.545225 132.266322)
-		(end 106.483909 132.205006)
-		(width 0.2)
-		(layer "F.Cu")
-		(net 36)
-	)
-	(segment
 		(start 125.28 133)
 		(end 123 133)
@@
 	)
 	(segment
+		(start 107.125 132.275)
+		(end 107.009624 132.159624)
+		(width 0.2)
+		(layer "F.Cu")
+		(net 36)
+	)
+	(segment
 		(start 108.962 134.288)
 		(end 109.375 134.701)
@@
 	)
 	(segment
+		(start 107.125 132.275)
+		(end 107.116322 132.266322)
+		(width 0.2)
+		(layer "F.Cu")
+		(net 36)
+	)
+	(segment
 		(start 159.275 105.6)
 		(end 159.275 105.295)
@@
 	)
 	(segment
-		(start 106.545225 132.266322)
-		(end 106.483909 132.205006)
-		(width 0.2)
-		(layer "F.Cu")
-		(net 36)
-	)
-	(segment
 		(start 138 110.465811)
 		(end 138.834189 111.3)
@@
 	)
 	(via
-		(at 106.545225 132.266322)
+		(at 107.125 132.275)
 		(size 0.45)
 		(drill 0.2)
@@
 	)
 	(segment
-		(start 104.875 128.325)
+		(start 105.174059 127.599492)
 		(end 104.875 127.898551)
 		(width 0.2)
@@
 	)
 	(segment
-		(start 104.875 127.898551)
-		(end 105.118132 127.655419)
+		(start 105.118132 127.656361)
+		(end 105.118132 127.65646)
 		(width 0.2)
 		(layer "F.Cu")
@@
 	)
 	(segment
-		(start 105.118132 127.655419)
-		(end 105.118132 127.65646)
+		(start 105.175001 127.599492)
+		(end 105.174059 127.599492)
+		(width 0.2)
+		(layer "F.Cu")
+		(net 99)
+	)
+	(segment
+		(start 105.175001 127.599492)
+		(end 105.118132 127.656361)
 		(width 0.2)
 		(layer "F.Cu")
@@
 		(net 99)
 	)
+	(segment
+		(start 104.875 127.898551)
+		(end 104.875 128.325)
+		(width 0.2)
+		(layer "F.Cu")
+		(net 99)
+	)
 	(via
-		(at 105.118132 127.655419)
+		(at 105.175001 127.599492)
 		(size 0.6)
 		(drill 0.3)
@@
 	)
 	(segment
-		(start 119 106.2)
-		(end 111.7671 106.2)
+		(start 108.668949 100.75)
+		(end 110.2873 102.368351)
 		(width 0.2)
 		(layer "In2.Cu")
@@
 	)
 	(segment
-		(start 120.6 107.8)
-		(end 119 106.2)
+		(start 105.062205 127.599492)
+		(end 104.599 127.136287)
 		(width 0.2)
 		(layer "In2.Cu")
@@
 	)
 	(segment
-		(start 104.599 124.789663)
-		(end 104.599 127.136287)
+		(start 105.175001 127.599492)
+		(end 105.062205 127.599492)
 		(width 0.2)
 		(layer "In2.Cu")
@@
 	)
 	(segment
-		(start 104.804763 106.054763)
+		(start 104.599 124.789663)
 		(end 104.804763 124.5839)
 		(width 0.2)
@@
 	(segment
 		(start 104.804763 124.5839)
-		(end 104.599 124.789663)
+		(end 104.804763 106.054763)
 		(width 0.2)
 		(layer "In2.Cu")
@@
 	)
 	(segment
-		(start 111.7671 106.2)
-		(end 110.2873 104.7202)
+		(start 103.1137 101.518451)
+		(end 103.882151 100.75)
 		(width 0.2)
 		(layer "In2.Cu")
@@
 	)
 	(segment
-		(start 103.1137 101.518451)
+		(start 104.804763 106.054763)
 		(end 103.1137 104.3637)
 		(width 0.2)
@@
 	)
 	(segment
-		(start 110.2873 104.7202)
-		(end 110.2873 102.368351)
+		(start 120.6 107.8)
+		(end 120.6 108.3)
+		(width 0.2)
+		(layer "In2.Cu")
+		(net 99)
+	)
+	(segment
+		(start 110.2873 102.368351)
+		(end 110.2873 104.7202)
 		(width 0.2)
 		(layer "In2.Cu")
@@
 	(segment
 		(start 103.1137 104.3637)
-		(end 104.804763 106.054763)
+		(end 103.1137 101.518451)
 		(width 0.2)
 		(layer "In2.Cu")
@@
 	)
 	(segment
-		(start 120.6 108.3)
+		(start 119 106.2)
 		(end 120.6 107.8)
 		(width 0.2)
@@
 	)
 	(segment
-		(start 104.599 127.136287)
-		(end 105.118132 127.655419)
+		(start 110.2873 104.7202)
+		(end 111.7671 106.2)
 		(width 0.2)
 		(layer "In2.Cu")
@@
 	(segment
 		(start 103.882151 100.75)
-		(end 103.1137 101.518451)
+		(end 108.668949 100.75)
 		(width 0.2)
 		(layer "In2.Cu")
@@
 	)
 	(segment
-		(start 110.2873 102.368351)
-		(end 108.668949 100.75)
+		(start 104.599 127.136287)
+		(end 104.599 124.789663)
 		(width 0.2)
 		(layer "In2.Cu")
@@
 	)
 	(segment
-		(start 108.668949 100.75)
-		(end 103.882151 100.75)
+		(start 111.7671 106.2)
+		(end 119 106.2)
 		(width 0.2)
 		(layer "In2.Cu")

Commit message: real_order2
Routing:
- net /SPI2_GPIO2: track 80.4 -> 79.9 mm
Changed lines of the file:
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@@
 	)
 	(segment
-		(start 129.052009 133.515091)
-		(end 129.052009 134)
+		(start 131.6661 130.901)
+		(end 129.052009 133.515091)
 		(width 0.2)
 		(layer "B.Cu")
@@
 		(end 108.8936 120.2686)
 		(width 0.5)
+		(layer "B.Cu")
+		(net 90)
+	)
+	(segment
+		(start 143.250565 130.500565)
+		(end 140.566535 130.500565)
+		(width 0.2)
 		(layer "B.Cu")
 		(net 90)
@@
 	)
 	(segment
-		(start 131.6661 130.901)
-		(end 129.052009 133.515091)
-		(width 0.2)
-		(layer "B.Cu")
-		(net 90)
-	)
-	(segment
-		(start 140.471476 130.901)
+		(start 154.864214 131.2)
+		(end 156.957107 133.292893)
+		(width 0.35)
+		(layer "B.Cu")
+		(net 90)
+	)
+	(segment
+		(start 140.1661 130.901)
 		(end 131.6661 130.901)
 		(width 0.2)
+		(layer "B.Cu")
+		(net 90)
+	)
+	(segment
+		(start 108.125 110.125)
+		(end 108.125 111.75)
+		(width 0.5)
+		(layer "B.Cu")
+		(net 90)
+	)
+	(segment
+		(start 108.8936 120.2686)
+		(end 108.8936 123.1436)
+		(width 0.5)
+		(layer "B.Cu")
+		(net 90)
+	)
+	(segment
+		(start 105.75 107.75)
+		(end 108.125 110.125)
+		(width 0.5)
+		(layer "B.Cu")
+		(net 90)
+	)
+	(segment
+		(start 140.566535 130.500565)
+		(end 140.1661 130.901)
+		(width 0.2)
+		(layer "B.Cu")
+		(net 90)
+	)
+	(segment
+		(start 114.249998 127.489498)
+		(end 111.6095 124.849)
+		(width 0.5)
+		(layer "B.Cu")
+		(net 90)
+	)
+	(segment
+		(start 154.864214 129.964214)
+		(end 154.864214 131.2)
+		(width 0.35)
+		(layer "B.Cu")
+		(net 90)
+	)
+	(segment
+		(start 111.9115 125.151)
+		(end 111.6095 124.849)
+		(width 0.5)
+		(layer "B.Cu")
+		(net 90)
+	)
+	(segment
+		(start 106 113.875)
+		(end 106 117.375)
+		(width 0.5)
+		(layer "B.Cu")
+		(net 90)
+	)
+	(segment
+		(start 109.75 124)
+		(end 110.7605 124)
+		(width 0.5)
+		(layer "B.Cu")
+		(net 90)
+	)
+	(segment
+		(start 154 129.1)
+		(end 154.864214 129.964214)
+		(width 0.35)
 		(layer "B.Cu")
 		(net 90)
@@
 	)
 	(segment
-		(start 154.864214 131.2)
-		(end 156.957107 133.292893)
-		(width 0.35)
-		(layer "B.Cu")
-		(net 90)
-	)
-	(segment
-		(start 108.125 110.125)
-		(end 108.125 111.75)
-		(width 0.5)
-		(layer "B.Cu")
-		(net 90)
-	)
-	(segment
-		(start 108.8936 120.2686)
-		(end 108.8936 123.1436)
-		(width 0.5)
-		(layer "B.Cu")
-		(net 90)
-	)
-	(segment
-		(start 105.75 107.75)
-		(end 108.125 110.125)
-		(width 0.5)
-		(layer "B.Cu")
-		(net 90)
-	)
-	(segment
-		(start 114.249998 127.489498)
-		(end 111.6095 124.849)
-		(width 0.5)
-		(layer "B.Cu")
-		(net 90)
-	)
-	(segment
-		(start 154.864214 129.964214)
-		(end 154.864214 131.2)
-		(width 0.35)
-		(layer "B.Cu")
-		(net 90)
-	)
-	(segment
-		(start 111.9115 125.151)
-		(end 111.6095 124.849)
-		(width 0.5)
-		(layer "B.Cu")
-		(net 90)
-	)
-	(segment
-		(start 106 113.875)
-		(end 106 117.375)
-		(width 0.5)
-		(layer "B.Cu")
-		(net 90)
-	)
-	(segment
-		(start 109.75 124)
-		(end 110.7605 124)
-		(width 0.5)
-		(layer "B.Cu")
-		(net 90)
-	)
-	(segment
-		(start 154 129.1)
-		(end 154.864214 129.964214)
-		(width 0.35)
-		(layer "B.Cu")
-		(net 90)
-	)
-	(segment
-		(start 143.250565 130.500565)
-		(end 140.871911 130.500565)
-		(width 0.2)
-		(layer "B.Cu")
-		(net 90)
-	)
-	(segment
 		(start 108.125 111.75)
 		(end 106 113.875)
@@
 		(end 146.55 129.1)
 		(width 0.35)
-		(layer "B.Cu")
-		(net 90)
-	)
-	(segment
-		(start 140.871911 130.500565)
-		(end 140.471476 130.901)
-		(width 0.2)
 		(layer "B.Cu")
 		(net 90)
@@
 		(end 139.651 109.5)
 		(width 0.3)
+		(layer "B.Cu")
+		(net 90)
+	)
+	(segment
+		(start 129.052009 133.515091)
+		(end 129.052009 134)
+		(width 0.2)
 		(layer "B.Cu")
 		(net 90)
@@
 	(segment
 		(start 102.99753 132.151)
-		(end 102.813439 131.966909)
+		(end 105.401 132.151)
+		(width 0.2)
+		(layer "B.Cu")
+		(net 93)
+	)
+	(segment
+		(start 141.825 128.675)
+		(end 141.825 126.175)
+		(width 0.2)
+		(layer "B.Cu")
+		(net 93)
+	)
+	(segment
+		(start 106.351692 133.101692)
+		(end 128.898308 133.101692)
+		(width 0.2)
+		(layer "B.Cu")
+		(net 93)
+	)
+	(segment
+		(start 102.813439 131.966909)
+		(end 102.99753 132.151)
 		(width 0.2)
 		(layer "B.Cu")
@@
 	(segment
 		(start 140 130.5)
+		(end 141.825 128.675)
+		(width 0.2)
+		(layer "B.Cu")
+		(net 93)
+	)
+	(segment
+		(start 128.898308 133.101692)
 		(end 131.5 130.5)
 		(width 0.2)
@@
 	(segment
 		(start 105.401 132.151)
-		(end 102.99753 132.151)
-		(width 0.2)
-		(layer "B.Cu")
-		(net 93)
-	)
-	(segment
-		(start 106.351692 133.101692)
-		(end 105.401 132.151)
-		(width 0.2)
-		(layer "B.Cu")
-		(net 93)
-	)
-	(segment
-		(start 142.5 126.85)
-		(end 142.5 128)
-		(width 0.2)
-		(layer "B.Cu")
-		(net 93)
-	)
-	(segment
-		(start 142.5 128)
+		(end 106.351692 133.101692)
+		(width 0.2)
+		(layer "B.Cu")
+		(net 93)
+	)
+	(segment
+		(start 141.825 126.175)
+		(end 141.4 125.75)
+		(width 0.2)
+		(layer "B.Cu")
+		(net 93)
+	)
+	(segment
+		(start 131.5 130.5)
 		(end 140 130.5)
 		(width 0.2)
 		(layer "B.Cu")
-		(net 93)
-	)
-	(segment
-		(start 141.4 125.75)
-		(end 142.5 126.85)
-		(width 0.2)
-		(layer "B.Cu")
-		(net 93)
-	)
-	(segment
-		(start 128.898308 133.101692)
-		(end 106.351692 133.101692)
-		(width 0.2)
-		(layer "B.Cu")
-		(net 93)
-	)
-	(segment
-		(start 131.5 130.5)
-		(end 128.898308 133.101692)
-		(width 0.2)
-		(layer "B.Cu")
