File: Board/MouseWB5.kicad_pcb (KiCad board)
At the start: 6 copper layers, 65.5 x 40 mm, 96 parts, among them J1 USB_C_Receptacle_USB2.0_14P, J9 Conn_01x02_Socket, M1 Conn_01x02_Socket, M2 Conn_01x02_Socket, M3 Conn_01x02_Socket, M4 Conn_01x02_Socket, M5 Conn_01x02_Socket, Q2 MCC SI8810, SW1 SW_Push, U1 STM32WB5MMG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

Commit message: real_order2
Routing:
- net Net-(LED8-DOUT): track 69.3 -> 67.8 mm
Changed lines of the file:
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@@
 	)
 	(segment
-		(start 155.25 128.25)
-		(end 158 131)
-		(width 0.2)
-		(layer "In2.Cu")
-		(net 21)
-	)
-	(segment
-		(start 158.37132 131.87868)
-		(end 158.37132 131.87132)
+		(start 155 126.5)
+		(end 155 128.5)
 		(width 0.2)
 		(layer "In2.Cu")
@@
 	)
 	(segment
-		(start 155.25 126.75)
-		(end 155.25 128.25)
+		(start 151.498 122.998)
+		(end 155 126.5)
 		(width 0.2)
 		(layer "In2.Cu")
@@
 	)
 	(segment
-		(start 151.498 122.8151)
-		(end 151.5 122.8171)
-		(width 0.2)
-		(layer "In2.Cu")
-		(net 21)
-	)
-	(segment
-		(start 151.5 122.8171)
-		(end 151.5 123)
-		(width 0.2)
-		(layer "In2.Cu")
-		(net 21)
-	)
-	(segment
-		(start 151.5 123)
-		(end 155.25 126.75)
-		(width 0.2)
-		(layer "In2.Cu")
-		(net 21)
-	)
-	(segment
 		(start 151.498 117.048066)
-		(end 151.498 122.8151)
+		(end 151.498 122.998)
 		(width 0.2)
 		(layer "In2.Cu")
@@
 	(segment
 		(start 158.37132 131.87132)
-		(end 158 131.5)
+		(end 158.37132 131.87868)
 		(width 0.2)
 		(layer "In2.Cu")
@@
 	)
 	(segment
-		(start 158 131.5)
-		(end 158 131)
+		(start 155 128.5)
+		(end 158.37132 131.87132)
 		(width 0.2)
 		(layer "In2.Cu")
@@
 	)
 	(segment
-		(start 148.90855 111.65855)
-		(end 150.40855 111.65855)
+		(start 151 112.25)
+		(end 151 114.582725)
 		(width 0.2)
 		(layer "In2.Cu")
@@
 	)
 	(segment
-		(start 156.5 126.5)
-		(end 156.5 127.25)
+		(start 152.5 116.082724)
+		(end 152.5 122.5)
 		(width 0.2)
 		(layer "In2.Cu")
@@
 	)
 	(segment
-		(start 152.5 122.5)
-		(end 156.5 126.5)
+		(start 156.5 127.25)
+		(end 159.714466 130.464466)
 		(width 0.2)
 		(layer "In2.Cu")
@@
 	)
 	(segment
-		(start 159.714466 130.464466)
-		(end 159.785534 130.464466)
+		(start 152.5 122.5)
+		(end 156.5 126.5)
 		(width 0.2)
 		(layer "In2.Cu")
@@
 	)
 	(segment
-		(start 152.5 116.082724)
-		(end 152.5 122.5)
+		(start 156.5 126.5)
+		(end 156.5 127.25)
 		(width 0.2)
 		(layer "In2.Cu")
@@
 	)
 	(segment
-		(start 150.40855 111.65855)
-		(end 151 112.25)
+		(start 151 114.582725)
+		(end 152.5 116.082724)
 		(width 0.2)
 		(layer "In2.Cu")
@@
 	)
 	(segment
-		(start 146.75 113.8171)
-		(end 148.90855 111.65855)
+		(start 146.75 120.051528)
+		(end 146.75 113.8171)
 		(width 0.2)
 		(layer "In2.Cu")
@@
 	)
 	(segment
-		(start 146.75 120.051528)
-		(end 146.75 113.8171)
+		(start 147.474236 120.775764)
+		(end 146.75 120.051528)
 		(width 0.2)
 		(layer "In2.Cu")
@@
 	)
 	(segment
-		(start 151 112.25)
-		(end 151 114.582725)
+		(start 150.40855 111.65855)
+		(end 151 112.25)
 		(width 0.2)
 		(layer "In2.Cu")
@@
 	)
 	(segment
-		(start 147.474236 120.775764)
-		(end 146.75 120.051528)
+		(start 148.90855 111.65855)
+		(end 150.40855 111.65855)
 		(width 0.2)
 		(layer "In2.Cu")
@@
 	)
 	(segment
-		(start 156.5 127.25)
-		(end 159.714466 130.464466)
+		(start 146.75 113.8171)
+		(end 148.90855 111.65855)
 		(width 0.2)
 		(layer "In2.Cu")
@@
 	)
 	(segment
-		(start 151 114.582725)
-		(end 152.5 116.082724)
+		(start 159.714466 130.464466)
+		(end 159.785534 130.464466)
 		(width 0.2)
 		(layer "In2.Cu")
@@
 	)
 	(segment
-		(start 105.062205 127.599492)
-		(end 104.599 127.136287)
+		(start 104.804763 106.054763)
+		(end 103.1137 104.3637)
 		(width 0.2)
 		(layer "In2.Cu")
@@
 	)
 	(segment
-		(start 104.599 124.789663)
-		(end 104.804763 124.5839)
+		(start 103.882151 100.75)
+		(end 108.668949 100.75)
 		(width 0.2)
 		(layer "In2.Cu")
@@
 	)
 	(segment
-		(start 104.804763 124.5839)
-		(end 104.804763 106.054763)
+		(start 105.062205 127.599492)
+		(end 104.599 127.136287)
 		(width 0.2)
 		(layer "In2.Cu")
@@
 	)
 	(segment
-		(start 103.1137 101.518451)
-		(end 103.882151 100.75)
+		(start 104.804763 124.5839)
+		(end 104.804763 106.054763)
 		(width 0.2)
 		(layer "In2.Cu")
@@
 	)
 	(segment
-		(start 104.804763 106.054763)
-		(end 103.1137 104.3637)
+		(start 119.3 106.5)
+		(end 120.6 107.8)
 		(width 0.2)
 		(layer "In2.Cu")
@@
 	)
 	(segment
-		(start 120.6 107.8)
-		(end 120.6 108.3)
+		(start 110.2873 102.368351)
+		(end 110.2873 104.7202)
 		(width 0.2)
 		(layer "In2.Cu")
@@
 	)
 	(segment
-		(start 110.2873 102.368351)
-		(end 110.2873 104.7202)
+		(start 110.2873 104.7202)
+		(end 112.0671 106.5)
 		(width 0.2)
 		(layer "In2.Cu")
@@
 	)
 	(segment
-		(start 119 106.2)
-		(end 120.6 107.8)
+		(start 120.6 107.8)
+		(end 120.6 108.3)
 		(width 0.2)
 		(layer "In2.Cu")
@@
 	)
 	(segment
-		(start 110.2873 104.7202)
-		(end 111.7671 106.2)
+		(start 103.1137 101.518451)
+		(end 103.882151 100.75)
 		(width 0.2)
 		(layer "In2.Cu")
@@
 	)
 	(segment
-		(start 103.882151 100.75)
-		(end 108.668949 100.75)
+		(start 104.599 127.136287)
+		(end 104.599 124.789663)
 		(width 0.2)
 		(layer "In2.Cu")
@@
 	)
 	(segment
-		(start 104.599 127.136287)
-		(end 104.599 124.789663)
+		(start 112.0671 106.5)
+		(end 119.3 106.5)
 		(width 0.2)
 		(layer "In2.Cu")
@@
 	)
 	(segment
-		(start 111.7671 106.2)
-		(end 119 106.2)
+		(start 104.599 124.789663)
+		(end 104.804763 124.5839)
 		(width 0.2)
 		(layer "In2.Cu")
@@
 	)
 	(segment
-		(start 157.5502 102.6502)
-		(end 157.1252 102.6502)
-		(width 0.2)
-		(layer "F.Cu")
-		(net 109)
-	)
-	(segment
-		(start 154.2 106.8)
-		(end 154.2 109.4)
-		(width 0.2)
-		(layer "F.Cu")
-		(net 109)
-	)
-	(segment
-		(start 112.926232 109.947)
-		(end 112.427232 109.448)
+		(start 105.948 109.448)
+		(end 105.5 109)
 		(width 0.2)
 		(layer "F.Cu")
@@
 	)
 	(segment
-		(start 139.345379 112.449)
-		(end 136.843379 109.947)
+		(start 105.5 106.57483)
+		(end 103.67247 104.7473)
 		(width 0.2)
 		(layer "F.Cu")
@@
 	)
 	(segment
-		(start 143.69104 112.449)
-		(end 139.345379 112.449)
+		(start 156.8 102.9754)
+		(end 156.8 104.549942)
 		(width 0.2)
 		(layer "F.Cu")
@@
 	)
 	(segment
-		(start 103.67247 104.7473)
-		(end 103.609451 104.7473)
+		(start 103.1137 104.251549)
+		(end 103.1137 102.3117)
 		(width 0.2)
 		(layer "F.Cu")
@@
 	)
 	(segment
-		(start 153.64632 109.95368)
-		(end 146.18636 109.95368)
+		(start 155.899 105.101)
+		(end 151.04632 109.95368)
 		(width 0.2)
 		(layer "F.Cu")
@@
 	)
 	(segment
-		(start 105.5 109)
-		(end 105.5 106.57483)
+		(start 156.8 104.549942)
+		(end 156.248942 105.101)
 		(width 0.2)
 		(layer "F.Cu")
@@
 	)
 	(segment
-		(start 156.8 104.549942)
-		(end 156.248942 105.101)
+		(start 103.609451 104.7473)
+		(end 103.1137 104.251549)
 		(width 0.2)
 		(layer "F.Cu")
@@
 	)
 	(segment
-		(start 154.2 109.4)
-		(end 153.64632 109.95368)
+		(start 103.1137 102.3117)
+		(end 102.1271 101.3251)
 		(width 0.2)
 		(layer "F.Cu")
@@
 	)
 	(segment
-		(start 105.5 106.57483)
-		(end 103.67247 104.7473)
+		(start 139.345379 112.449)
+		(end 136.843379 109.947)
 		(width 0.2)
 		(layer "F.Cu")
@@
 	)
 	(segment
-		(start 157.1252 102.6502)
-		(end 156.8 102.9754)
+		(start 112.427232 109.448)
+		(end 105.948 109.448)
 		(width 0.2)
 		(layer "F.Cu")
@@
 	)
 	(segment
-		(start 103.1137 104.251549)
-		(end 103.1137 102.3117)
+		(start 143.69104 112.449)
+		(end 139.345379 112.449)
 		(width 0.2)
 		(layer "F.Cu")
@@
 	)
 	(segment
-		(start 105.948 109.448)
-		(end 105.5 109)
+		(start 156.248942 105.101)
+		(end 155.899 105.101)
 		(width 0.2)
 		(layer "F.Cu")
@@
 	)
 	(segment
-		(start 102.1271 101.3251)
-		(end 101.9247 101.3251)
+		(start 112.926232 109.947)
+		(end 112.427232 109.448)
 		(width 0.2)
 		(layer "F.Cu")
@@
 	)
 	(segment
-		(start 155.899 105.101)
-		(end 154.2 106.8)
+		(start 105.5 109)
+		(end 105.5 106.57483)
 		(width 0.2)
 		(layer "F.Cu")
@@
 	)
 	(segment
-		(start 103.609451 104.7473)
-		(end 103.1137 104.251549)
+		(start 151.04632 109.95368)
+		(end 146.18636 109.95368)
 		(width 0.2)
 		(layer "F.Cu")
@@
 	)
 	(segment
-		(start 112.427232 109.448)
-		(end 105.948 109.448)
+		(start 103.67247 104.7473)
+		(end 103.609451 104.7473)
 		(width 0.2)
 		(layer "F.Cu")
@@
 	)
 	(segment
-		(start 156.248942 105.101)
-		(end 155.899 105.101)
+		(start 102.1271 101.3251)
+		(end 101.9247 101.3251)
 		(width 0.2)
 		(layer "F.Cu")
@@
 	)
 	(segment
-		(start 156.8 102.9754)
-		(end 156.8 104.549942)
+		(start 157.5502 102.6502)
+		(end 157.1252 102.6502)
 		(width 0.2)
 		(layer "F.Cu")
@@
 	)
 	(segment
-		(start 103.1137 102.3117)
-		(end 102.1271 101.3251)
+		(start 157.1252 102.6502)
+		(end 156.8 102.9754)
 		(width 0.2)
 		(layer "F.Cu")
